File: Electrical/Nova/Barometer.sch (KiCad schematic (older format))
At the start: 2 parts

Commit message: Fixed Power Supply
Parts:
- Barometer201: symbol MS560702BA03-50:MS560702BA03-50 -> Nova-rescue:MS560702BA03-50-MS560702BA03-50
Changed lines of the file:
@@
 $EndDescr
 $Comp
-L MS560702BA03-50:MS560702BA03-50 Barometer201
+L Nova-rescue:MS560702BA03-50-MS560702BA03-50 Barometer201
 U 1 1 5F01D3E2
 P 6000 3600

Commit message: Added Gyroscope
Parts:
- Barometer201: symbol Nova-rescue:MS560702BA03-50-MS560702BA03-50 -> Nova-rescue:MS560702BA03-50-MS560702BA03-50-Nova-rescue
Changed lines of the file:
@@
 $Descr A4 11693 8268
 encoding utf-8
-Sheet 10 13
+Sheet 10 14
 Title ""
 Date ""
@@
 $EndDescr
 $Comp
-L Nova-rescue:MS560702BA03-50-MS560702BA03-50 Barometer201
+L Nova-rescue:MS560702BA03-50-MS560702BA03-50-Nova-rescue Barometer201
 U 1 1 5F01D3E2
 P 6000 3600

Commit message: Added Gyro pins. Organized Schematic
Need to determine if we need the interrupt pins for the sensors.
Parts:
- Barometer201: symbol Nova-rescue:MS560702BA03-50-MS560702BA03-50-Nova-rescue -> Nova-rescue:MS560702BA03-50-MS560702BA03-50-Nova-rescue-Nova-rescue
Changed lines of the file:
@@
 $EndDescr
 $Comp
-L Nova-rescue:MS560702BA03-50-MS560702BA03-50-Nova-rescue Barometer201
+L Nova-rescue:MS560702BA03-50-MS560702BA03-50-Nova-rescue-Nova-rescue Barometer201
 U 1 1 5F01D3E2
 P 6000 3600

Commit message: Added Pyro Channels
Parts:
- Barometer201: symbol Nova-rescue:MS560702BA03-50-MS560702BA03-50-Nova-rescue-Nova-rescue -> Nova-rescue:MS560702BA03-50-MS560702BA03-50-Nova-rescue-Nova-rescue-Nova-rescue
Changed lines of the file:
@@
 $Descr A4 11693 8268
 encoding utf-8
-Sheet 10 14
+Sheet 10 16
 Title ""
 Date ""
@@
 $EndDescr
 $Comp
-L Nova-rescue:MS560702BA03-50-MS560702BA03-50-Nova-rescue-Nova-rescue Barometer201
+L Nova-rescue:MS560702BA03-50-MS560702BA03-50-Nova-rescue-Nova-rescue-Nova-rescue Barometer201
 U 1 1 5F01D3E2
 P 6000 3600

Commit message: Added LED sheet and pins
Parts:
- Barometer201: symbol Nova-rescue:MS560702BA03-50-MS560702BA03-50-Nova-rescue-Nova-rescue-Nova-rescue -> Nova-rescue:MS560702BA03-50-MS560702BA03-50-Nova-rescue-Nova-rescue-Nova-rescue-Nova-rescue
Changed lines of the file:
@@
 $Descr A4 11693 8268
 encoding utf-8
-Sheet 10 16
+Sheet 10 18
 Title ""
 Date ""
@@
 $EndDescr
 $Comp
-L Nova-rescue:MS560702BA03-50-MS560702BA03-50-Nova-rescue-Nova-rescue-Nova-rescue Barometer201
+L Nova-rescue:MS560702BA03-50-MS560702BA03-50-Nova-rescue-Nova-rescue-Nova-rescue-Nova-rescue Barometer201
 U 1 1 5F01D3E2
 P 6000 3600

Commit message: Minor update
Parts:
- C801: renamed from C201; footprint Capacitor_SMD:C_0805_2012Metric_Pad1.15x1.40mm_HandSolder -> NOVA MCU (STM):C_0805_2012Metric
- renumbered Barometer201 to Barometer801
Changed lines of the file:
@@
 $Descr A4 11693 8268
 encoding utf-8
-Sheet 10 18
+Sheet 8 18
 Title ""
 Date ""
@@
 $EndDescr
 $Comp
-L Nova-rescue:MS560702BA03-50-MS560702BA03-50-Nova-rescue-Nova-rescue-Nova-rescue-Nova-rescue Barometer201
+L Nova-rescue:MS560702BA03-50-MS560702BA03-50-Nova-rescue-Nova-rescue-Nova-rescue-Nova-rescue Barometer?
 U 1 1 5F01D3E2
 P 6000 3600
-AR Path="/5F01D3E2" Ref="Barometer201"  Part="1"
-AR Path="/5F013144/5F01D3E2" Ref="Barometer201"  Part="1"
-AR Path="/5F3A063C/5F01D3E2" Ref="Barometer201"  Part="1"
-F 0 "Barometer201" H 6000 4187 60  0000 C CNN
+AR Path="/5F01D3E2" Ref="Barometer?"  Part="1"
+AR Path="/5F013144/5F01D3E2" Ref="Barometer?"  Part="1"
+AR Path="/5F3A063C/5F01D3E2" Ref="Barometer801"  Part="1"
+F 0 "Barometer801" H 6000 4187 60  0000 C CNN
 F 1 "MS560702BA03-50" H 6000 4081 60  0000 C CNN
 F 2 "Footprint Library:MS560702BA03-50" H 6000 4040 60  0001 C CNN
@@
 $EndComp
 $Comp
-L power:+3V3 #PWR0201
+L power:+3V3 #PWR0801
 U 1 1 5F01D3E8
 P 4450 3300
-F 0 "#PWR0201" H 4450 3150 50  0001 C CNN
+F 0 "#PWR0801" H 4450 3150 50  0001 C CNN
 F 1 "+3V3" H 4465 3473 50  0000 C CNN
 F 2 "" H 4450 3300 50  0001 C CNN
@@
 $EndComp
 $Comp
-L pspice:C C201
+L pspice:C C801
 U 1 1 5F01D3EE
 P 4450 3750
-F 0 "C201" H 4628 3796 50  0000 L CNN
+F 0 "C801" H 4628 3796 50  0000 L CNN
 F 1 "100nF" H 4628 3705 50  0000 L CNN
-F 2 "Capacitor_SMD:C_0805_2012Metric_Pad1.15x1.40mm_HandSolder" H 4450 3750 50  0001 C CNN
+F 2 "NOVA MCU (STM):C_0805_2012Metric" H 4450 3750 50  0001 C CNN
 F 3 "~" H 4450 3750 50  0001 C CNN
 	1    4450 3750
@@
 	4450 4000 4450 4100
 $Comp
-L power:GND #PWR0202
+L power:GND #PWR0802
 U 1 1 5F01D3F6
 P 4450 4150
-F 0 "#PWR0202" H 4450 3900 50  0001 C CNN
+F 0 "#PWR0802" H 4450 3900 50  0001 C CNN
 F 1 "GND" H 4455 3977 50  0000 C CNN
 F 2 "" H 4450 4150 50  0001 C CNN

Commit message: Added Accelerometer
Parts:
- Barometer801: symbol Nova-rescue:MS560702BA03-50-MS560702BA03-50-Nova-rescue-Nova-rescue-Nova-rescue-Nova-rescue -> Nova-rescue:MS560702BA03-50-MS560702BA03-50-Nova-rescue-Nova-rescue-Nova-rescue-Nova-rescue-Nova-rescue
Changed lines of the file:
@@
 $Descr A4 11693 8268
 encoding utf-8
-Sheet 8 18
+Sheet 8 19
 Title ""
 Date ""
@@
 $EndDescr
 $Comp
-L Nova-rescue:MS560702BA03-50-MS560702BA03-50-Nova-rescue-Nova-rescue-Nova-rescue-Nova-rescue Barometer?
+L Nova-rescue:MS560702BA03-50-MS560702BA03-50-Nova-rescue-Nova-rescue-Nova-rescue-Nova-rescue-Nova-rescue Barometer?
 U 1 1 5F01D3E2
 P 6000 3600
