File: Electrical/Nova/Clocks.sch (KiCad schematic (older format))
At the start: 7 parts

Commit message: Added Barometer, Flash, SD, and Power Supply
Parts:
- C401, C402, C403, C404: symbol Nova_Microcontroller:C -> Nova-rescue:C-Nova_Microcontroller
- R?: symbol Nova_Microcontroller:R_US -> Nova-rescue:R_US-Nova_Microcontroller
- Y?: symbol Nova_Microcontroller:Crystal_GND24 -> Nova-rescue:Crystal_GND24-Nova_Microcontroller
- Y?: symbol Nova_Microcontroller:Crystal -> Nova-rescue:Crystal-Nova_Microcontroller
Changed lines of the file:
@@
 $Descr A4 11693 8268
 encoding utf-8
-Sheet 6 9
+Sheet 6 13
 Title "Microcontroller"
 Date "2020-07-02"
@@
 $EndBitmap
 $Comp
-L Nova_Microcontroller:Crystal_GND24 Y?
+L Nova-rescue:Crystal_GND24-Nova_Microcontroller Y?
 U 1 1 5EE6B82C
 P 3350 3550
@@
 	3350 3350 3350 3150
 $Comp
-L Nova_Microcontroller:Crystal Y?
+L Nova-rescue:Crystal-Nova_Microcontroller Y?
 U 1 1 5EE717EC
 P 8050 3550
@@
 	3350 3850 3700 3850
 $Comp
-L Nova_Microcontroller:C C?
+L Nova-rescue:C-Nova_Microcontroller C?
 U 1 1 5EE74A4A
 P 7600 3700
@@
 $EndComp
 $Comp
-L Nova_Microcontroller:C C?
+L Nova-rescue:C-Nova_Microcontroller C?
 U 1 1 5EE7523E
 P 8550 3700
@@
 	2600 3550 2450 3550
 $Comp
-L Nova_Microcontroller:R_US R?
+L Nova-rescue:R_US-Nova_Microcontroller R?
 U 1 1 5EE707DE
 P 2750 3550
@@
 $EndBitmap
 $Comp
-L Nova_Microcontroller:C C?
+L Nova-rescue:C-Nova_Microcontroller C?
 U 1 1 5EE74215
 P 3700 3700
@@
 $EndComp
 $Comp
-L Nova_Microcontroller:C C?
+L Nova-rescue:C-Nova_Microcontroller C?
 U 1 1 5EE73815
 P 3000 3700

Commit message: Fixed Power Supply
Parts:
- C401, C402, C403, C404: symbol Nova-rescue:C-Nova_Microcontroller -> Nova-rescue:C-Nova_Microcontroller-Nova-rescue
- R?: symbol Nova-rescue:R_US-Nova_Microcontroller -> Nova-rescue:R_US-Nova_Microcontroller-Nova-rescue
- Y?: symbol Nova-rescue:Crystal_GND24-Nova_Microcontroller -> Nova-rescue:Crystal_GND24-Nova_Microcontroller-Nova-rescue
- Y?: symbol Nova-rescue:Crystal-Nova_Microcontroller -> Nova-rescue:Crystal-Nova_Microcontroller-Nova-rescue
Changed lines of the file:
@@
 $EndBitmap
 $Comp
-L Nova-rescue:Crystal_GND24-Nova_Microcontroller Y?
+L Nova-rescue:Crystal_GND24-Nova_Microcontroller-Nova-rescue Y?
 U 1 1 5EE6B82C
 P 3350 3550
@@
 	3350 3350 3350 3150
 $Comp
-L Nova-rescue:Crystal-Nova_Microcontroller Y?
+L Nova-rescue:Crystal-Nova_Microcontroller-Nova-rescue Y?
 U 1 1 5EE717EC
 P 8050 3550
@@
 	3350 3850 3700 3850
 $Comp
-L Nova-rescue:C-Nova_Microcontroller C?
+L Nova-rescue:C-Nova_Microcontroller-Nova-rescue C?
 U 1 1 5EE74A4A
 P 7600 3700
@@
 $EndComp
 $Comp
-L Nova-rescue:C-Nova_Microcontroller C?
+L Nova-rescue:C-Nova_Microcontroller-Nova-rescue C?
 U 1 1 5EE7523E
 P 8550 3700
@@
 	2600 3550 2450 3550
 $Comp
-L Nova-rescue:R_US-Nova_Microcontroller R?
+L Nova-rescue:R_US-Nova_Microcontroller-Nova-rescue R?
 U 1 1 5EE707DE
 P 2750 3550
@@
 $EndBitmap
 $Comp
-L Nova-rescue:C-Nova_Microcontroller C?
+L Nova-rescue:C-Nova_Microcontroller-Nova-rescue C?
 U 1 1 5EE74215
 P 3700 3700
@@
 $EndComp
 $Comp
-L Nova-rescue:C-Nova_Microcontroller C?
+L Nova-rescue:C-Nova_Microcontroller-Nova-rescue C?
 U 1 1 5EE73815
 P 3000 3700

Commit message: Added Gyroscope
Parts:
- C401, C402, C403, C404: symbol Nova-rescue:C-Nova_Microcontroller-Nova-rescue -> Nova-rescue:C-Nova_Microcontroller-Nova-rescue-Nova-rescue
- R?: symbol Nova-rescue:R_US-Nova_Microcontroller-Nova-rescue -> Nova-rescue:R_US-Nova_Microcontroller-Nova-rescue-Nova-rescue
- Y?: symbol Nova-rescue:Crystal_GND24-Nova_Microcontroller-Nova-rescue -> Nova-rescue:Crystal_GND24-Nova_Microcontroller-Nova-rescue-Nova-rescue
- Y?: symbol Nova-rescue:Crystal-Nova_Microcontroller-Nova-rescue -> Nova-rescue:Crystal-Nova_Microcontroller-Nova-rescue-Nova-rescue
Changed lines of the file:
@@
 $Descr A4 11693 8268
 encoding utf-8
-Sheet 6 13
+Sheet 6 14
 Title "Microcontroller"
 Date "2020-07-02"
@@
 $EndBitmap
 $Comp
-L Nova-rescue:Crystal_GND24-Nova_Microcontroller-Nova-rescue Y?
+L Nova-rescue:Crystal_GND24-Nova_Microcontroller-Nova-rescue-Nova-rescue Y?
 U 1 1 5EE6B82C
 P 3350 3550
@@
 	3350 3350 3350 3150
 $Comp
-L Nova-rescue:Crystal-Nova_Microcontroller-Nova-rescue Y?
+L Nova-rescue:Crystal-Nova_Microcontroller-Nova-rescue-Nova-rescue Y?
 U 1 1 5EE717EC
 P 8050 3550
@@
 	3350 3850 3700 3850
 $Comp
-L Nova-rescue:C-Nova_Microcontroller-Nova-rescue C?
+L Nova-rescue:C-Nova_Microcontroller-Nova-rescue-Nova-rescue C?
 U 1 1 5EE74A4A
 P 7600 3700
@@
 $EndComp
 $Comp
-L Nova-rescue:C-Nova_Microcontroller-Nova-rescue C?
+L Nova-rescue:C-Nova_Microcontroller-Nova-rescue-Nova-rescue C?
 U 1 1 5EE7523E
 P 8550 3700
@@
 	2600 3550 2450 3550
 $Comp
-L Nova-rescue:R_US-Nova_Microcontroller-Nova-rescue R?
+L Nova-rescue:R_US-Nova_Microcontroller-Nova-rescue-Nova-rescue R?
 U 1 1 5EE707DE
 P 2750 3550
@@
 $EndBitmap
 $Comp
-L Nova-rescue:C-Nova_Microcontroller-Nova-rescue C?
+L Nova-rescue:C-Nova_Microcontroller-Nova-rescue-Nova-rescue C?
 U 1 1 5EE74215
 P 3700 3700
@@
 $EndComp
 $Comp
-L Nova-rescue:C-Nova_Microcontroller-Nova-rescue C?
+L Nova-rescue:C-Nova_Microcontroller-Nova-rescue-Nova-rescue C?
 U 1 1 5EE73815
 P 3000 3700

Commit message: Added Gyro pins. Organized Schematic
Need to determine if we need the interrupt pins for the sensors.
Parts:
- C401, C402, C403, C404: symbol Nova-rescue:C-Nova_Microcontroller-Nova-rescue-Nova-rescue -> Nova-rescue:C-Nova_Microcontroller-Nova-rescue-Nova-rescue-Nova-rescue
- R?: symbol Nova-rescue:R_US-Nova_Microcontroller-Nova-rescue-Nova-rescue -> Nova-rescue:R_US-Nova_Microcontroller-Nova-rescue-Nova-rescue-Nova-rescue
- Y?: symbol Nova-rescue:Crystal_GND24-Nova_Microcontroller-Nova-rescue-Nova-rescue -> Nova-rescue:Crystal_GND24-Nova_Microcontroller-Nova-rescue-Nova-rescue-Nova-rescue
- Y?: symbol Nova-rescue:Crystal-Nova_Microcontroller-Nova-rescue-Nova-rescue -> Nova-rescue:Crystal-Nova_Microcontroller-Nova-rescue-Nova-rescue-Nova-rescue
Changed lines of the file:
@@
 $EndBitmap
 $Comp
-L Nova-rescue:Crystal_GND24-Nova_Microcontroller-Nova-rescue-Nova-rescue Y?
+L Nova-rescue:Crystal_GND24-Nova_Microcontroller-Nova-rescue-Nova-rescue-Nova-rescue Y?
 U 1 1 5EE6B82C
 P 3350 3550
@@
 	3350 3350 3350 3150
 $Comp
-L Nova-rescue:Crystal-Nova_Microcontroller-Nova-rescue-Nova-rescue Y?
+L Nova-rescue:Crystal-Nova_Microcontroller-Nova-rescue-Nova-rescue-Nova-rescue Y?
 U 1 1 5EE717EC
 P 8050 3550
@@
 	3350 3850 3700 3850
 $Comp
-L Nova-rescue:C-Nova_Microcontroller-Nova-rescue-Nova-rescue C?
+L Nova-rescue:C-Nova_Microcontroller-Nova-rescue-Nova-rescue-Nova-rescue C?
 U 1 1 5EE74A4A
 P 7600 3700
@@
 $EndComp
 $Comp
-L Nova-rescue:C-Nova_Microcontroller-Nova-rescue-Nova-rescue C?
+L Nova-rescue:C-Nova_Microcontroller-Nova-rescue-Nova-rescue-Nova-rescue C?
 U 1 1 5EE7523E
 P 8550 3700
@@
 	2600 3550 2450 3550
 $Comp
-L Nova-rescue:R_US-Nova_Microcontroller-Nova-rescue-Nova-rescue R?
+L Nova-rescue:R_US-Nova_Microcontroller-Nova-rescue-Nova-rescue-Nova-rescue R?
 U 1 1 5EE707DE
 P 2750 3550
@@
 $EndBitmap
 $Comp
-L Nova-rescue:C-Nova_Microcontroller-Nova-rescue-Nova-rescue C?
+L Nova-rescue:C-Nova_Microcontroller-Nova-rescue-Nova-rescue-Nova-rescue C?
 U 1 1 5EE74215
 P 3700 3700
@@
 $EndComp
 $Comp
-L Nova-rescue:C-Nova_Microcontroller-Nova-rescue-Nova-rescue C?
+L Nova-rescue:C-Nova_Microcontroller-Nova-rescue-Nova-rescue-Nova-rescue C?
 U 1 1 5EE73815
 P 3000 3700

Commit message: Added Pyro Channels
Parts:
- C401, C402, C403, C404: symbol Nova-rescue:C-Nova_Microcontroller-Nova-rescue-Nova-rescue-Nova-rescue -> Nova-rescue:C-Nova_Microcontroller-Nova-rescue-Nova-rescue-Nova-rescue-Nova-rescue
- R?: symbol Nova-rescue:R_US-Nova_Microcontroller-Nova-rescue-Nova-rescue-Nova-rescue -> Nova-rescue:R_US-Nova_Microcontroller-Nova-rescue-Nova-rescue-Nova-rescue-Nova-rescue
- Y?: symbol Nova-rescue:Crystal_GND24-Nova_Microcontroller-Nova-rescue-Nova-rescue-Nova-rescue -> Nova-rescue:Crystal_GND24-Nova_Microcontroller-Nova-rescue-Nova-rescue-Nova-rescue-Nova-rescue
- Y?: symbol Nova-rescue:Crystal-Nova_Microcontroller-Nova-rescue-Nova-rescue-Nova-rescue -> Nova-rescue:Crystal-Nova_Microcontroller-Nova-rescue-Nova-rescue-Nova-rescue-Nova-rescue
Changed lines of the file:
@@
 $Descr A4 11693 8268
 encoding utf-8
-Sheet 6 14
+Sheet 6 16
 Title "Microcontroller"
 Date "2020-07-02"
@@
 $EndBitmap
 $Comp
-L Nova-rescue:Crystal_GND24-Nova_Microcontroller-Nova-rescue-Nova-rescue-Nova-rescue Y?
+L Nova-rescue:Crystal_GND24-Nova_Microcontroller-Nova-rescue-Nova-rescue-Nova-rescue-Nova-rescue Y?
 U 1 1 5EE6B82C
 P 3350 3550
@@
 	3350 3350 3350 3150
 $Comp
-L Nova-rescue:Crystal-Nova_Microcontroller-Nova-rescue-Nova-rescue-Nova-rescue Y?
+L Nova-rescue:Crystal-Nova_Microcontroller-Nova-rescue-Nova-rescue-Nova-rescue-Nova-rescue Y?
 U 1 1 5EE717EC
 P 8050 3550
@@
 	3350 3850 3700 3850
 $Comp
-L Nova-rescue:C-Nova_Microcontroller-Nova-rescue-Nova-rescue-Nova-rescue C?
+L Nova-rescue:C-Nova_Microcontroller-Nova-rescue-Nova-rescue-Nova-rescue-Nova-rescue C?
 U 1 1 5EE74A4A
 P 7600 3700
@@
 $EndComp
 $Comp
-L Nova-rescue:C-Nova_Microcontroller-Nova-rescue-Nova-rescue-Nova-rescue C?
+L Nova-rescue:C-Nova_Microcontroller-Nova-rescue-Nova-rescue-Nova-rescue-Nova-rescue C?
 U 1 1 5EE7523E
 P 8550 3700
@@
 	2600 3550 2450 3550
 $Comp
-L Nova-rescue:R_US-Nova_Microcontroller-Nova-rescue-Nova-rescue-Nova-rescue R?
+L Nova-rescue:R_US-Nova_Microcontroller-Nova-rescue-Nova-rescue-Nova-rescue-Nova-rescue R?
 U 1 1 5EE707DE
 P 2750 3550
@@
 $EndBitmap
 $Comp
-L Nova-rescue:C-Nova_Microcontroller-Nova-rescue-Nova-rescue-Nova-rescue C?
+L Nova-rescue:C-Nova_Microcontroller-Nova-rescue-Nova-rescue-Nova-rescue-Nova-rescue C?
 U 1 1 5EE74215
 P 3700 3700
@@
 $EndComp
 $Comp
-L Nova-rescue:C-Nova_Microcontroller-Nova-rescue-Nova-rescue-Nova-rescue C?
+L Nova-rescue:C-Nova_Microcontroller-Nova-rescue-Nova-rescue-Nova-rescue-Nova-rescue C?
 U 1 1 5EE73815
 P 3000 3700

Commit message: Added LED sheet and pins
Parts:
- C401, C402, C403, C404: symbol Nova-rescue:C-Nova_Microcontroller-Nova-rescue-Nova-rescue-Nova-rescue-Nova-rescue -> Nova-rescue:C-Nova_Microcontroller-Nova-rescue-Nova-rescue-Nova-rescue-Nova-rescue-Nova-rescue
- R?: symbol Nova-rescue:R_US-Nova_Microcontroller-Nova-rescue-Nova-rescue-Nova-rescue-Nova-rescue -> Nova-rescue:R_US-Nova_Microcontroller-Nova-rescue-Nova-rescue-Nova-rescue-Nova-rescue-Nova-rescue
- Y?: symbol Nova-rescue:Crystal_GND24-Nova_Microcontroller-Nova-rescue-Nova-rescue-Nova-rescue-Nova-rescue -> Nova-rescue:Crystal_GND24-Nova_Microcontroller-Nova-rescue-Nova-rescue-Nova-rescue-Nova-rescue-Nova-rescue
- Y?: symbol Nova-rescue:Crystal-Nova_Microcontroller-Nova-rescue-Nova-rescue-Nova-rescue-Nova-rescue -> Nova-rescue:Crystal-Nova_Microcontroller-Nova-rescue-Nova-rescue-Nova-rescue-Nova-rescue-Nova-rescue
Changed lines of the file:
@@
 $Descr A4 11693 8268
 encoding utf-8
-Sheet 6 16
+Sheet 6 18
 Title "Microcontroller"
 Date "2020-07-02"
@@
 $EndBitmap
 $Comp
-L Nova-rescue:Crystal_GND24-Nova_Microcontroller-Nova-rescue-Nova-rescue-Nova-rescue-Nova-rescue Y?
+L Nova-rescue:Crystal_GND24-Nova_Microcontroller-Nova-rescue-Nova-rescue-Nova-rescue-Nova-rescue-Nova-rescue Y?
 U 1 1 5EE6B82C
 P 3350 3550
@@
 	3350 3350 3350 3150
 $Comp
-L Nova-rescue:Crystal-Nova_Microcontroller-Nova-rescue-Nova-rescue-Nova-rescue-Nova-rescue Y?
+L Nova-rescue:Crystal-Nova_Microcontroller-Nova-rescue-Nova-rescue-Nova-rescue-Nova-rescue-Nova-rescue Y?
 U 1 1 5EE717EC
 P 8050 3550
@@
 	3350 3850 3700 3850
 $Comp
-L Nova-rescue:C-Nova_Microcontroller-Nova-rescue-Nova-rescue-Nova-rescue-Nova-rescue C?
+L Nova-rescue:C-Nova_Microcontroller-Nova-rescue-Nova-rescue-Nova-rescue-Nova-rescue-Nova-rescue C?
 U 1 1 5EE74A4A
 P 7600 3700
@@
 $EndComp
 $Comp
-L Nova-rescue:C-Nova_Microcontroller-Nova-rescue-Nova-rescue-Nova-rescue-Nova-rescue C?
+L Nova-rescue:C-Nova_Microcontroller-Nova-rescue-Nova-rescue-Nova-rescue-Nova-rescue-Nova-rescue C?
 U 1 1 5EE7523E
 P 8550 3700
@@
 	2600 3550 2450 3550
 $Comp
-L Nova-rescue:R_US-Nova_Microcontroller-Nova-rescue-Nova-rescue-Nova-rescue-Nova-rescue R?
+L Nova-rescue:R_US-Nova_Microcontroller-Nova-rescue-Nova-rescue-Nova-rescue-Nova-rescue-Nova-rescue R?
 U 1 1 5EE707DE
 P 2750 3550
@@
 $EndBitmap
 $Comp
-L Nova-rescue:C-Nova_Microcontroller-Nova-rescue-Nova-rescue-Nova-rescue-Nova-rescue C?
+L Nova-rescue:C-Nova_Microcontroller-Nova-rescue-Nova-rescue-Nova-rescue-Nova-rescue-Nova-rescue C?
 U 1 1 5EE74215
 P 3700 3700
@@
 $EndComp
 $Comp
-L Nova-rescue:C-Nova_Microcontroller-Nova-rescue-Nova-rescue-Nova-rescue-Nova-rescue C?
+L Nova-rescue:C-Nova_Microcontroller-Nova-rescue-Nova-rescue-Nova-rescue-Nova-rescue-Nova-rescue C?
 U 1 1 5EE73815
 P 3000 3700

Commit message: Minor update
Parts:
- C401, C402, C403, C404: footprint NOVA MCU (STM):C_0805_2012Metric_Pad1.15x1.40mm_HandSolder -> NOVA MCU (STM):C_0805_2012Metric
- gave numbers to parts that had none: 3
Connections:
- net CLOCKIN: now also C402.1
- net RTCCRYSTALIN: now also C404.1
- net RTCCRYSTALOUT: now also C403.1
- net at R401.1, Y401.1: now also C401.1
Changed lines of the file:
@@
 $Descr A4 11693 8268
 encoding utf-8
-Sheet 6 18
+Sheet 4 18
 Title "Microcontroller"
 Date "2020-07-02"
@@
 $EndBitmap
 $Comp
-L Nova-rescue:Crystal_GND24-Nova_Microcontroller-Nova-rescue-Nova-rescue-Nova-rescue-Nova-rescue-Nova-rescue Y?
+L Nova-rescue:Crystal_GND24-Nova_Microcontroller-Nova-rescue-Nova-rescue-Nova-rescue-Nova-rescue-Nova-rescue Y401
 U 1 1 5EE6B82C
 P 3350 3550
-F 0 "Y?" H 3300 4300 50  0000 L CNN
+F 0 "Y401" H 3300 4300 50  0000 L CNN
 F 1 "ECS-260-8-36B-CKY-TR" H 2850 4200 50  0000 L CNN
 F 2 "NOVA MCU (STM):ECX-2236B" H 3350 3550 50  0001 C CNN
@@
 CLOCKOUT
 $Comp
-L power:GND #PWR?
+L power:GND #PWR0402
 U 1 1 5EE6F36D
 P 3350 3950
-F 0 "#PWR?" H 3350 3700 50  0001 C CNN
+F 0 "#PWR0402" H 3350 3700 50  0001 C CNN
 F 1 "GND" H 3355 3777 50  0000 C CNN
 F 2 "" H 3350 3950 50  0001 C CNN
@@
 $EndComp
 $Comp
-L power:GND #PWR?
+L power:GND #PWR0401
 U 1 1 5EE6FC19
 P 3350 3150
-F 0 "#PWR?" H 3350 2900 50  0001 C CNN
+F 0 "#PWR0401" H 3350 2900 50  0001 C CNN
 F 1 "GND" H 3355 2977 50  0000 C CNN
 F 2 "" H 3350 3150 50  0001 C CNN
@@
 	3350 3350 3350 3150
 $Comp
-L Nova-rescue:Crystal-Nova_Microcontroller-Nova-rescue-Nova-rescue-Nova-rescue-Nova-rescue-Nova-rescue Y?
+L Nova-rescue:Crystal-Nova_Microcontroller-Nova-rescue-Nova-rescue-Nova-rescue-Nova-rescue-Nova-rescue Y402
 U 1 1 5EE717EC
 P 8050 3550
-F 0 "Y?" H 8050 3818 50  0000 C CNN
+F 0 "Y402" H 8050 3818 50  0000 C CNN
 F 1 "JTX310" H 8050 3727 50  0000 C CNN
 F 2 "NOVA MCU (STM):JTX310" H 8050 3550 50  0001 C CNN
@@
 P 7600 3700
 AR Path="/5EE74A4A" Ref="C?"  Part="1"
-AR Path="/5EE654BB/5EE655E0/5EE74A4A" Ref="C403"  Part="1"
+AR Path="/5EE654BB/5EE655E0/5EE74A4A" Ref="C?"  Part="1"
 AR Path="/5F319C9C/5EE74A4A" Ref="C403"  Part="1"
 F 0 "C403" H 7715 3746 50  0000 L CNN
 F 1 "18pf" H 7715 3655 50  0000 L CNN
-F 2 "NOVA MCU (STM):C_0805_2012Metric_Pad1.15x1.40mm_HandSolder" H 7638 3550 50  0001 C CNN
+F 2 "NOVA MCU (STM):C_0805_2012Metric" H 7638 3550 50  0001 C CNN
 F 3 "~" H 7600 3700 50  0001 C CNN
 	1    7600 3700
@@
 P 8550 3700
 AR Path="/5EE7523E" Ref="C?"  Part="1"
-AR Path="/5EE654BB/5EE655E0/5EE7523E" Ref="C404"  Part="1"
+AR Path="/5EE654BB/5EE655E0/5EE7523E" Ref="C?"  Part="1"
 AR Path="/5F319C9C/5EE7523E" Ref="C404"  Part="1"
 F 0 "C404" H 8665 3746 50  0000 L CNN
 F 1 "18pf" H 8665 3655 50  0000 L CNN
-F 2 "NOVA MCU (STM):C_0805_2012Metric_Pad1.15x1.40mm_HandSolder" H 8588 3550 50  0001 C CNN
+F 2 "NOVA MCU (STM):C_0805_2012Metric" H 8588 3550 50  0001 C CNN
 F 3 "~" H 8550 3700 50  0001 C CNN
 	1    8550 3700
@@
 	7600 3850 8100 3850
 $Comp
-L power:GND #PWR?
+L power:GND #PWR0403
 U 1 1 5EE75B51
 P 8100 3850
-F 0 "#PWR?" H 8100 3600 50  0001 C CNN
+F 0 "#PWR0403" H 8100 3600 50  0001 C CNN
 F 1 "GND" H 8105 3677 50  0000 C CNN
 F 2 "" H 8100 3850 50  0001 C CNN
@@
 	2600 3550 2450 3550
 $Comp
-L Nova-rescue:R_US-Nova_Microcontroller-Nova-rescue-Nova-rescue-Nova-rescue-Nova-rescue-Nova-rescue R?
+L Nova-rescue:R_US-Nova_Microcontroller-Nova-rescue-Nova-rescue-Nova-rescue-Nova-rescue-Nova-rescue R401
 U 1 1 5EE707DE
 P 2750 3550
-F 0 "R?" V 2545 3550 50  0000 C CNN
+F 0 "R401" V 2545 3550 50  0000 C CNN
 F 1 "TBD" V 2636 3550 50  0000 C CNN
 F 2 "NOVA MCU (STM):R_0805_2012Metric_Pad1.15x1.40mm_HandSolder" V 2790 3540 50  0001 C CNN
@@
 P 3700 3700
 AR Path="/5EE74215" Ref="C?"  Part="1"
-AR Path="/5EE654BB/5EE655E0/5EE74215" Ref="C402"  Part="1"
+AR Path="/5EE654BB/5EE655E0/5EE74215" Ref="C?"  Part="1"
 AR Path="/5F319C9C/5EE74215" Ref="C402"  Part="1"
 F 0 "C402" H 3815 3746 50  0000 L CNN
 F 1 "10pf" H 3815 3655 50  0000 L CNN
-F 2 "NOVA MCU (STM):C_0805_2012Metric_Pad1.15x1.40mm_HandSolder" H 3738 3550 50  0001 C CNN
+F 2 "NOVA MCU (STM):C_0805_2012Metric" H 3738 3550 50  0001 C CNN
 F 3 "~" H 3700 3700 50  0001 C CNN
 	1    3700 3700
@@
 P 3000 3700
 AR Path="/5EE73815" Ref="C?"  Part="1"
-AR Path="/5EE654BB/5EE655E0/5EE73815" Ref="C401"  Part="1"
+AR Path="/5EE654BB/5EE655E0/5EE73815" Ref="C?"  Part="1"
 AR Path="/5F319C9C/5EE73815" Ref="C401"  Part="1"
 F 0 "C401" H 2700 3750 50  0000 L CNN
 F 1 "10pf" H 2700 3650 50  0000 L CNN
-F 2 "NOVA MCU (STM):C_0805_2012Metric_Pad1.15x1.40mm_HandSolder" H 3038 3550 50  0001 C CNN
+F 2 "NOVA MCU (STM):C_0805_2012Metric" H 3038 3550 50  0001 C CNN
 F 3 "~" H 3000 3700 50  0001 C CNN
 	1    3000 3700
@@
 $EndComp
 Wire Wire Line
-	3500 3550 3900 3550
+	3500 3550 3700 3550
 Wire Wire Line
-	7200 3550 7900 3550
+	7200 3550 7600 3550
 Wire Wire Line
-	8200 3550 9050 3550
+	8200 3550 8550 3550
 Wire Wire Line
-	2900 3550 3200 3550
+	2900 3550 3000 3550
+Connection ~ 3000 3550
+Wire Wire Line
+	3000 3550 3200 3550
+Connection ~ 3700 3550
+Wire Wire Line
+	3700 3550 3900 3550
+Connection ~ 7600 3550
+Wire Wire Line
+	7600 3550 7900 3550
+Connection ~ 8550 3550
+Wire Wire Line
+	8550 3550 9050 3550
 $EndSCHEMATC

Commit message: Added Accelerometer
Parts:
- C401, C402, C403, C404: symbol Nova-rescue:C-Nova_Microcontroller-Nova-rescue-Nova-rescue-Nova-rescue-Nova-rescue-Nova-rescue -> Nova-rescue:C-Nova_Microcontroller-Nova-rescue-Nova-rescue-Nova-rescue-Nova-rescue-Nova-rescue-Nova-rescue
- R401: symbol Nova-rescue:R_US-Nova_Microcontroller-Nova-rescue-Nova-rescue-Nova-rescue-Nova-rescue-Nova-rescue -> Nova-rescue:R_US-Nova_Microcontroller-Nova-rescue-Nova-rescue-Nova-rescue-Nova-rescue-Nova-rescue-Nova-rescue
- Y401: symbol Nova-rescue:Crystal_GND24-Nova_Microcontroller-Nova-rescue-Nova-rescue-Nova-rescue-Nova-rescue-Nova-rescue -> Nova-rescue:Crystal_GND24-Nova_Microcontroller-Nova-rescue-Nova-rescue-Nova-rescue-Nova-rescue-Nova-rescue-Nova-rescue
- Y402: symbol Nova-rescue:Crystal-Nova_Microcontroller-Nova-rescue-Nova-rescue-Nova-rescue-Nova-rescue-Nova-rescue -> Nova-rescue:Crystal-Nova_Microcontroller-Nova-rescue-Nova-rescue-Nova-rescue-Nova-rescue-Nova-rescue-Nova-rescue
Changed lines of the file:
@@
 $Descr A4 11693 8268
 encoding utf-8
-Sheet 4 18
+Sheet 4 19
 Title "Microcontroller"
 Date "2020-07-02"
@@
 $EndBitmap
 $Comp
-L Nova-rescue:Crystal_GND24-Nova_Microcontroller-Nova-rescue-Nova-rescue-Nova-rescue-Nova-rescue-Nova-rescue Y401
+L Nova-rescue:Crystal_GND24-Nova_Microcontroller-Nova-rescue-Nova-rescue-Nova-rescue-Nova-rescue-Nova-rescue-Nova-rescue Y401
 U 1 1 5EE6B82C
 P 3350 3550
@@
 	3350 3350 3350 3150
 $Comp
-L Nova-rescue:Crystal-Nova_Microcontroller-Nova-rescue-Nova-rescue-Nova-rescue-Nova-rescue-Nova-rescue Y402
+L Nova-rescue:Crystal-Nova_Microcontroller-Nova-rescue-Nova-rescue-Nova-rescue-Nova-rescue-Nova-rescue-Nova-rescue Y402
 U 1 1 5EE717EC
 P 8050 3550
@@
 	3350 3850 3700 3850
 $Comp
-L Nova-rescue:C-Nova_Microcontroller-Nova-rescue-Nova-rescue-Nova-rescue-Nova-rescue-Nova-rescue C?
+L Nova-rescue:C-Nova_Microcontroller-Nova-rescue-Nova-rescue-Nova-rescue-Nova-rescue-Nova-rescue-Nova-rescue C?
 U 1 1 5EE74A4A
 P 7600 3700
@@
 $EndComp
 $Comp
-L Nova-rescue:C-Nova_Microcontroller-Nova-rescue-Nova-rescue-Nova-rescue-Nova-rescue-Nova-rescue C?
+L Nova-rescue:C-Nova_Microcontroller-Nova-rescue-Nova-rescue-Nova-rescue-Nova-rescue-Nova-rescue-Nova-rescue C?
 U 1 1 5EE7523E
 P 8550 3700
@@
 	2600 3550 2450 3550
 $Comp
-L Nova-rescue:R_US-Nova_Microcontroller-Nova-rescue-Nova-rescue-Nova-rescue-Nova-rescue-Nova-rescue R401
+L Nova-rescue:R_US-Nova_Microcontroller-Nova-rescue-Nova-rescue-Nova-rescue-Nova-rescue-Nova-rescue-Nova-rescue R401
 U 1 1 5EE707DE
 P 2750 3550
@@
 $EndBitmap
 $Comp
-L Nova-rescue:C-Nova_Microcontroller-Nova-rescue-Nova-rescue-Nova-rescue-Nova-rescue-Nova-rescue C?
+L Nova-rescue:C-Nova_Microcontroller-Nova-rescue-Nova-rescue-Nova-rescue-Nova-rescue-Nova-rescue-Nova-rescue C?
 U 1 1 5EE74215
 P 3700 3700
@@
 $EndComp
 $Comp
-L Nova-rescue:C-Nova_Microcontroller-Nova-rescue-Nova-rescue-Nova-rescue-Nova-rescue-Nova-rescue C?
+L Nova-rescue:C-Nova_Microcontroller-Nova-rescue-Nova-rescue-Nova-rescue-Nova-rescue-Nova-rescue-Nova-rescue C?
 U 1 1 5EE73815
 P 3000 3700
