File: Electrical/Nova/FlashChip.sch (KiCad schematic (older format))
At the start: 2 parts, among them U10 W25N512GVPIT

Commit message: Fixed Power Supply
Parts:
- U10: symbol Flash_Chip:W25N512GVPIT -> Nova-rescue:W25N512GVPIT-Flash_Chip
Changed lines of the file:
@@
 $EndComp
 $Comp
-L Flash_Chip:W25N512GVPIT U10
+L Nova-rescue:W25N512GVPIT-Flash_Chip U10
 U 1 1 5F01567A
 P 5450 3400
+AR Path="/5F01567A" Ref="U10"  Part="1"
+AR Path="/5F3B5C2E/5F01567A" Ref="U10"  Part="1"
 F 0 "U10" H 5450 3815 50  0000 C CNN
 F 1 "W25N512GVPIT" H 5450 3724 50  0000 C CNN

Commit message: Added Gyroscope
Parts:
- U10: symbol Nova-rescue:W25N512GVPIT-Flash_Chip -> Nova-rescue:W25N512GVPIT-Flash_Chip-Nova-rescue
Changed lines of the file:
@@
 $Descr A4 11693 8268
 encoding utf-8
-Sheet 13 13
+Sheet 13 14
 Title ""
 Date ""
@@
 $EndComp
 $Comp
-L Nova-rescue:W25N512GVPIT-Flash_Chip U10
+L Nova-rescue:W25N512GVPIT-Flash_Chip-Nova-rescue U10
 U 1 1 5F01567A
 P 5450 3400

Commit message: Added Gyro pins. Organized Schematic
Need to determine if we need the interrupt pins for the sensors.
Parts:
- U10: symbol Nova-rescue:W25N512GVPIT-Flash_Chip-Nova-rescue -> Nova-rescue:W25N512GVPIT-Flash_Chip-Nova-rescue-Nova-rescue
Changed lines of the file:
@@
 $EndComp
 $Comp
-L Nova-rescue:W25N512GVPIT-Flash_Chip-Nova-rescue U10
+L Nova-rescue:W25N512GVPIT-Flash_Chip-Nova-rescue-Nova-rescue U10
 U 1 1 5F01567A
 P 5450 3400

Commit message: Added Pyro Channels
Parts:
- U10: symbol Nova-rescue:W25N512GVPIT-Flash_Chip-Nova-rescue-Nova-rescue -> Nova-rescue:W25N512GVPIT-Flash_Chip-Nova-rescue-Nova-rescue-Nova-rescue
Changed lines of the file:
@@
 $Descr A4 11693 8268
 encoding utf-8
-Sheet 13 14
+Sheet 13 16
 Title ""
 Date ""
@@
 $EndComp
 $Comp
-L Nova-rescue:W25N512GVPIT-Flash_Chip-Nova-rescue-Nova-rescue U10
+L Nova-rescue:W25N512GVPIT-Flash_Chip-Nova-rescue-Nova-rescue-Nova-rescue U10
 U 1 1 5F01567A
 P 5450 3400

Commit message: Added LED sheet and pins
Parts:
- U10: symbol Nova-rescue:W25N512GVPIT-Flash_Chip-Nova-rescue-Nova-rescue-Nova-rescue -> Nova-rescue:W25N512GVPIT-Flash_Chip-Nova-rescue-Nova-rescue-Nova-rescue-Nova-rescue
Changed lines of the file:
@@
 $Descr A4 11693 8268
 encoding utf-8
-Sheet 13 16
+Sheet 13 18
 Title ""
 Date ""
@@
 $EndComp
 $Comp
-L Nova-rescue:W25N512GVPIT-Flash_Chip-Nova-rescue-Nova-rescue-Nova-rescue U10
+L Nova-rescue:W25N512GVPIT-Flash_Chip-Nova-rescue-Nova-rescue-Nova-rescue-Nova-rescue U10
 U 1 1 5F01567A
 P 5450 3400

Commit message: Minor update
Parts:
- C1101: renamed from C401; footprint Capacitor_SMD:C_0805_2012Metric_Pad1.15x1.40mm_HandSolder -> NOVA MCU (STM):C_0805_2012Metric
- renumbered U10 to U1101
Changed lines of the file:
@@
 $Descr A4 11693 8268
 encoding utf-8
-Sheet 13 18
+Sheet 11 18
 Title ""
 Date ""
@@
 	5100 3550 4850 3550
 $Comp
-L power:GND #PWR0401
+L power:GND #PWR01101
 U 1 1 5F0563D1
 P 4850 3550
-F 0 "#PWR0401" H 4850 3300 50  0001 C CNN
+F 0 "#PWR01101" H 4850 3300 50  0001 C CNN
 F 1 "GND" V 4855 3422 50  0000 R CNN
 F 2 "" H 4850 3550 50  0001 C CNN
@@
 $EndComp
 $Comp
-L power:+3.3V #PWR0402
+L power:+3.3V #PWR01103
 U 1 1 5F055C85
 P 6700 3250
-F 0 "#PWR0402" H 6700 3100 50  0001 C CNN
+F 0 "#PWR01103" H 6700 3100 50  0001 C CNN
 F 1 "+3.3V" V 6715 3378 50  0000 L CNN
 F 2 "" H 6700 3250 50  0001 C CNN
@@
 	6700 3250 6550 3250
 $Comp
-L Device:C C401
+L Device:C C1101
 U 1 1 5F06D2E9
 P 6550 3400
-F 0 "C401" V 6298 3400 50  0000 C CNN
+F 0 "C1101" V 6298 3400 50  0000 C CNN
 F 1 "100nF" V 6389 3400 50  0000 C CNN
-F 2 "Capacitor_SMD:C_0805_2012Metric_Pad1.15x1.40mm_HandSolder" H 6588 3250 50  0001 C CNN
+F 2 "NOVA MCU (STM):C_0805_2012Metric" H 6588 3250 50  0001 C CNN
 F 3 "~" H 6550 3400 50  0001 C CNN
 	1    6550 3400
@@
 $EndComp
 $Comp
-L Nova-rescue:W25N512GVPIT-Flash_Chip-Nova-rescue-Nova-rescue-Nova-rescue-Nova-rescue U10
+L Nova-rescue:W25N512GVPIT-Flash_Chip-Nova-rescue-Nova-rescue-Nova-rescue-Nova-rescue U?
 U 1 1 5F01567A
 P 5450 3400
-AR Path="/5F01567A" Ref="U10"  Part="1"
-AR Path="/5F3B5C2E/5F01567A" Ref="U10"  Part="1"
-F 0 "U10" H 5450 3815 50  0000 C CNN
+AR Path="/5F01567A" Ref="U?"  Part="1"
+AR Path="/5F3B5C2E/5F01567A" Ref="U1101"  Part="1"
+F 0 "U1101" H 5450 3815 50  0000 C CNN
 F 1 "W25N512GVPIT" H 5450 3724 50  0000 C CNN
 F 2 "Footprint Library:W25N512GVPIT" H 5450 3700 50  0001 C CNN
@@
 	6550 3550 6550 3700
 $Comp
-L power:GND #PWR0102
+L power:GND #PWR01102
 U 1 1 5F03FC8A
 P 6550 3700
-F 0 "#PWR0102" H 6550 3450 50  0001 C CNN
+F 0 "#PWR01102" H 6550 3450 50  0001 C CNN
 F 1 "GND" H 6555 3527 50  0000 C CNN
 F 2 "" H 6550 3700 50  0001 C CNN

Commit message: Added Accelerometer
Parts:
- U1101: symbol Nova-rescue:W25N512GVPIT-Flash_Chip-Nova-rescue-Nova-rescue-Nova-rescue-Nova-rescue -> Nova-rescue:W25N512GVPIT-Flash_Chip-Nova-rescue-Nova-rescue-Nova-rescue-Nova-rescue-Nova-rescue
Changed lines of the file:
@@
 $Descr A4 11693 8268
 encoding utf-8
-Sheet 11 18
+Sheet 11 19
 Title ""
 Date ""
@@
 $EndComp
 $Comp
-L Nova-rescue:W25N512GVPIT-Flash_Chip-Nova-rescue-Nova-rescue-Nova-rescue-Nova-rescue U?
+L Nova-rescue:W25N512GVPIT-Flash_Chip-Nova-rescue-Nova-rescue-Nova-rescue-Nova-rescue-Nova-rescue U?
 U 1 1 5F01567A
 P 5450 3400
