File: Electrical/Nova/MicroSD.sch (KiCad schematic (older format))
At the start: 2 parts

Commit message: Minor update
Parts:
- C1001: renamed from C301; footprint Capacitor_SMD:C_0805_2012Metric_Pad1.15x1.40mm_HandSolder -> NOVA MCU (STM):C_0805_2012Metric
- renumbered Micro_SD301 to Micro_SD1001
Changed lines of the file:
@@
 $Descr A4 11693 8268
 encoding utf-8
-Sheet 12 18
+Sheet 10 18
 Title ""
 Date ""
@@
 	5000 3650 4650 3650
 $Comp
-L power:GND #PWR0302
+L power:GND #PWR01003
 U 1 1 5F054581
 P 4650 3750
-F 0 "#PWR0302" H 4650 3500 50  0001 C CNN
+F 0 "#PWR01003" H 4650 3500 50  0001 C CNN
 F 1 "GND" V 4655 3622 50  0000 R CNN
 F 2 "" H 4650 3750 50  0001 C CNN
@@
 	5000 3350 4650 3350
 $Comp
-L Connector:Micro_SD_Card Micro_SD301
+L Connector:Micro_SD_Card Micro_SD1001
 U 1 1 5F05B5EB
 P 5900 3550
-F 0 "Micro_SD301" H 5850 4267 50  0000 C CNN
+F 0 "Micro_SD1001" H 5850 4267 50  0000 C CNN
 F 1 "Micro_SD_Card" H 5850 4176 50  0000 C CNN
 F 2 "Connector_Card:microSD_HC_Molex_104031-0811" H 7050 3850 50  0001 C CNN
@@
 P 3900 3550
 AR Path="/5F0430E6/5F04B12E/5F06F178" Ref="#PWR?"  Part="1"
-AR Path="/5F0430E6/5F04B2FC/5F06F178" Ref="#PWR0301"  Part="1"
-AR Path="/5F3B5BD1/5F06F178" Ref="#PWR0301"  Part="1"
-F 0 "#PWR0301" H 3900 3400 50  0001 C CNN
+AR Path="/5F0430E6/5F04B2FC/5F06F178" Ref="#PWR?"  Part="1"
+AR Path="/5F3B5BD1/5F06F178" Ref="#PWR01001"  Part="1"
+F 0 "#PWR01001" H 3900 3400 50  0001 C CNN
 F 1 "+3.3V" V 3915 3678 50  0000 L CNN
 F 2 "" H 3900 3550 50  0001 C CNN
@@
 P 4050 3700
 AR Path="/5F0430E6/5F04B12E/5F06F17E" Ref="C?"  Part="1"
-AR Path="/5F0430E6/5F04B2FC/5F06F17E" Ref="C301"  Part="1"
-AR Path="/5F3B5BD1/5F06F17E" Ref="C301"  Part="1"
-F 0 "C301" V 3798 3700 50  0000 C CNN
+AR Path="/5F0430E6/5F04B2FC/5F06F17E" Ref="C?"  Part="1"
+AR Path="/5F3B5BD1/5F06F17E" Ref="C1001"  Part="1"
+F 0 "C1001" V 3798 3700 50  0000 C CNN
 F 1 "100nF" V 3889 3700 50  0000 C CNN
-F 2 "Capacitor_SMD:C_0805_2012Metric_Pad1.15x1.40mm_HandSolder" H 4088 3550 50  0001 C CNN
+F 2 "NOVA MCU (STM):C_0805_2012Metric" H 4088 3550 50  0001 C CNN
 F 3 "~" H 4050 3700 50  0001 C CNN
 	1    4050 3700
@@
 Connection ~ 4050 3550
 $Comp
-L power:GND #PWR0101
+L power:GND #PWR01002
 U 1 1 5F03E8D8
 P 4050 4000
-F 0 "#PWR0101" H 4050 3750 50  0001 C CNN
+F 0 "#PWR01002" H 4050 3750 50  0001 C CNN
 F 1 "GND" H 4055 3827 50  0000 C CNN
 F 2 "" H 4050 4000 50  0001 C CNN
