File: Electrical/Nova/SWD.sch (KiCad schematic (older format))
At the start: 2 parts, among them J701 Conn_01x06_Male, J702 Conn_01x06_Male

Commit message: Fixed File paths for 0603
Parts:
- J701, J702: symbol Nova-rescue:Conn_01x06_Male-Nova_Microcontroller-Nova-rescue-Nova-rescue-Nova-rescue-Nova-rescue-Nova-rescue-Nova-rescue -> Nova-rescue:Conn_01x06_Male-Nova_Microcontroller-Nova-rescue-Nova-rescue-Nova-rescue-Nova-rescue-Nova-rescue-Nova-rescu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
Changed lines of the file:
@@
 $EndDescr
 $Comp
-L Nova-rescue:Conn_01x06_Male-Nova_Microcontroller-Nova-rescue-Nova-rescue-Nova-rescue-Nova-rescue-Nova-rescue-Nova-rescue J702
+L Nova-rescue:Conn_01x06_Male-Nova_Microcontroller-Nova-rescue-Nova-rescue-Nova-rescue-Nova-rescue-Nova-rescue-Nova-rescue-Nova-rescue J702
 U 1 1 5F3A5F38
 P 5150 3600
@@
 $EndBitmap
 $Comp
-L Nova-rescue:Conn_01x06_Male-Nova_Microcontroller-Nova-rescue-Nova-rescue-Nova-rescue-Nova-rescue-Nova-rescue-Nova-rescue J701
+L Nova-rescue:Conn_01x06_Male-Nova_Microcontroller-Nova-rescue-Nova-rescue-Nova-rescue-Nova-rescue-Nova-rescue-Nova-rescue-Nova-rescue J701
 U 1 1 5EF13F12
 P 5150 3600
