File: Electrical/Nova/USB-C.sch (KiCad schematic (older format))
At the start: 14 parts

Commit message: Added Barometer, Flash, SD, and Power Supply
Parts:
- C? (x4): symbol Nova_Microcontroller:C -> Nova-rescue:C-Nova_Microcontroller
- D?: symbol Nova_Microcontroller:LED -> Nova-rescue:LED-Nova_Microcontroller
- F?: symbol Nova_Microcontroller:Fuse -> Nova-rescue:Fuse-Nova_Microcontroller
- FB?: symbol Nova_Microcontroller:Ferrite_Bead -> Nova-rescue:Ferrite_Bead-Nova_Microcontroller
- J?: symbol Nova_Microcontroller:USB_C_Receptacle -> Nova-rescue:USB_C_Receptacle-Nova_Microcontroller
- R? (x5): symbol Nova_Microcontroller:R_US -> Nova-rescue:R_US-Nova_Microcontroller
- U?: symbol Nova_Microcontroller:FT234XD-R -> Nova-rescue:FT234XD-R-Nova_Microcontroller
Changed lines of the file:
@@
 $Descr A4 11693 8268
 encoding utf-8
-Sheet 5 9
+Sheet 5 13
 Title "Microcontroller"
 Date "2020-07-02"
@@
 $EndBitmap
 $Comp
-L Nova_Microcontroller:USB_C_Receptacle J?
+L Nova-rescue:USB_C_Receptacle-Nova_Microcontroller J?
 U 1 1 5EE7E0E1
 P 3900 3500
@@
 Connection ~ 3900 5300
 $Comp
-L Nova_Microcontroller:Fuse F?
+L Nova-rescue:Fuse-Nova_Microcontroller F?
 U 1 1 5EE8054D
 P 5050 2500
@@
 	4500 2500 4700 2500
 $Comp
-L Nova_Microcontroller:FT234XD-R U?
+L Nova-rescue:FT234XD-R-Nova_Microcontroller U?
 U 1 1 5EE8343B
 P 7900 3500
@@
 $EndComp
 $Comp
-L Nova_Microcontroller:Ferrite_Bead FB?
+L Nova-rescue:Ferrite_Bead-Nova_Microcontroller FB?
 U 1 1 5EE89DD0
 P 6050 2500
@@
 	6200 2500 8000 2500
 $Comp
-L Nova_Microcontroller:R_US R?
+L Nova-rescue:R_US-Nova_Microcontroller R?
 U 1 1 5EE8D72F
 P 5150 3000
@@
 	7250 3600 7500 3600
 $Comp
-L Nova_Microcontroller:C C?
+L Nova-rescue:C-Nova_Microcontroller C?
 U 1 1 5EE93320
 P 5950 3750
@@
 $EndComp
 $Comp
-L Nova_Microcontroller:C C?
+L Nova-rescue:C-Nova_Microcontroller C?
 U 1 1 5EE93CEE
 P 6400 3750
@@
 Connection ~ 6200 4050
 $Comp
-L Nova_Microcontroller:R_US R?
+L Nova-rescue:R_US-Nova_Microcontroller R?
 U 1 1 5EE8E4DE
 P 5150 3200
@@
 $EndComp
 $Comp
-L Nova_Microcontroller:C C?
+L Nova-rescue:C-Nova_Microcontroller C?
 U 1 1 5EE97E32
 P 9400 3650
@@
 	9400 3800 9400 3950
 $Comp
-L Nova_Microcontroller:C C?
+L Nova-rescue:C-Nova_Microcontroller C?
 U 1 1 5EE98E46
 P 5450 2350
@@
 	5450 2200 5450 2000
 $Comp
-L Nova_Microcontroller:LED D?
+L Nova-rescue:LED-Nova_Microcontroller D?
 U 1 1 5EE9CC36
 P 7150 4650
@@
 $EndComp
 $Comp
-L Nova_Microcontroller:R_US R?
+L Nova-rescue:R_US-Nova_Microcontroller R?
 U 1 1 5EE9D264
 P 6550 4650
@@
 D2+
 $Comp
-L Nova_Microcontroller:R_US R?
+L Nova-rescue:R_US-Nova_Microcontroller R?
 U 1 1 5EF2AE69
 P 6200 3000
@@
 $EndComp
 $Comp
-L Nova_Microcontroller:R_US R?
+L Nova-rescue:R_US-Nova_Microcontroller R?
 U 1 1 5EF2B785
 P 6450 2750

Commit message: Fixed Power Supply
Parts:
- removed C?: 47pF, NOVA MCU (STM):C_0805_2012Metric_Pad1.15x1.40mm_HandSolder, symbol Nova-rescue:C-Nova_Microcontroller
- removed C?: 100nF, NOVA MCU (STM):C_0805_2012Metric_Pad1.15x1.40mm_HandSolder, symbol Nova-rescue:C-Nova_Microcontroller
- removed FB?: 600 OHM, NOVA MCU (STM):R_0805_2012Metric_Pad1.15x1.40mm_HandSolder, symbol Nova-rescue:Ferrite_Bead-Nova_Microcontroller
- removed R?: 5K, NOVA MCU (STM):R_0805_2012Metric_Pad1.15x1.40mm_HandSolder, symbol Nova-rescue:R_US-Nova_Microcontroller
- removed U?: FT234XD-R, NOVA MCU (STM):DFN-12-1EP_3x3mm, symbol Nova-rescue:FT234XD-R-Nova_Microcontroller
- added C?: 47pF, NOVA MCU (STM):C_0805_2012Metric_Pad1.15x1.40mm_HandSolder, symbol Nova-rescue:C-Nova_Microcontroller-Nova-rescue
- added C?: 100nF, NOVA MCU (STM):C_0805_2012Metric_Pad1.15x1.40mm_HandSolder, symbol Nova-rescue:C-Nova_Microcontroller-Nova-rescue
- added FB?: 600 OHM, NOVA MCU (STM):R_0805_2012Metric_Pad1.15x1.40mm_HandSolder, symbol Nova-rescue:Ferrite_Bead-Nova_Microcontroller-Nova-rescue
- added R?: 5K, NOVA MCU (STM):R_0805_2012Metric_Pad1.15x1.40mm_HandSolder, symbol Nova-rescue:R_US-Nova_Microcontroller-Nova-rescue
- added U?: FT234XD-R, NOVA MCU (STM):DFN-12-1EP_3x3mm, symbol Nova-rescue:FT234XD-R-Nova_Microcontroller-Nova-rescue
- C? (x2): symbol Nova-rescue:C-Nova_Microcontroller -> Nova-rescue:C-Nova_Microcontroller-Nova-rescue
- D?: symbol Nova-rescue:LED-Nova_Microcontroller -> Nova-rescue:LED-Nova_Microcontroller-Nova-rescue
- F?: symbol Nova-rescue:Fuse-Nova_Microcontroller -> Nova-rescue:Fuse-Nova_Microcontroller-Nova-rescue
- J?: symbol Nova-rescue:USB_C_Receptacle-Nova_Microcontroller -> Nova-rescue:USB_C_Receptacle-Nova_Microcontroller-Nova-rescue
- R? (x4): symbol Nova-rescue:R_US-Nova_Microcontroller -> Nova-rescue:R_US-Nova_Microcontroller-Nova-rescue
Changed lines of the file:
@@
 $Descr A4 11693 8268
 encoding utf-8
-Sheet 5 13
+Sheet 4 13
 Title "Microcontroller"
 Date "2020-07-02"
@@
 $EndBitmap
 $Comp
-L Nova-rescue:USB_C_Receptacle-Nova_Microcontroller J?
+L Nova-rescue:USB_C_Receptacle-Nova_Microcontroller-Nova-rescue J?
 U 1 1 5EE7E0E1
 P 3900 3500
@@
 $Comp
 L power:GND #PWR?
-U 1 1 5EE7F750
+U 1 1 5F3B6869
 P 3900 5300
 F 0 "#PWR?" H 3900 5050 50  0001 C CNN
@@
 Connection ~ 3900 5300
 $Comp
-L Nova-rescue:Fuse-Nova_Microcontroller F?
+L Nova-rescue:Fuse-Nova_Microcontroller-Nova-rescue F?
 U 1 1 5EE8054D
 P 5050 2500
@@
 	4500 2500 4700 2500
 $Comp
-L Nova-rescue:FT234XD-R-Nova_Microcontroller U?
-U 1 1 5EE8343B
+L Nova-rescue:FT234XD-R-Nova_Microcontroller-Nova-rescue U?
+U 1 1 5F3B686B
 P 7900 3500
 F 0 "U?" H 7450 4000 60  0000 C CNN
@@
 $EndComp
 $Comp
-L Nova-rescue:Ferrite_Bead-Nova_Microcontroller FB?
-U 1 1 5EE89DD0
+L Nova-rescue:Ferrite_Bead-Nova_Microcontroller-Nova-rescue FB?
+U 1 1 5F3B686C
 P 6050 2500
 F 0 "FB?" V 5776 2500 50  0000 C CNN
@@
 	6200 2500 8000 2500
 $Comp
-L Nova-rescue:R_US-Nova_Microcontroller R?
+L Nova-rescue:R_US-Nova_Microcontroller-Nova-rescue R?
 U 1 1 5EE8D72F
 P 5150 3000
@@
 $Comp
 L power:+3.3V #PWR?
-U 1 1 5EE9256E
+U 1 1 5F3B6871
 P 7250 3600
 F 0 "#PWR?" H 7250 3450 50  0001 C CNN
@@
 	7250 3600 7500 3600
 $Comp
-L Nova-rescue:C-Nova_Microcontroller C?
-U 1 1 5EE93320
+L Nova-rescue:C-Nova_Microcontroller-Nova-rescue C?
+U 1 1 5F3B6872
 P 5950 3750
 F 0 "C?" H 6065 3796 50  0000 L CNN
@@
 $EndComp
 $Comp
-L Nova-rescue:C-Nova_Microcontroller C?
+L Nova-rescue:C-Nova_Microcontroller-Nova-rescue C?
 U 1 1 5EE93CEE
 P 6400 3750
@@
 Connection ~ 6200 4050
 $Comp
-L Nova-rescue:R_US-Nova_Microcontroller R?
+L Nova-rescue:R_US-Nova_Microcontroller-Nova-rescue R?
 U 1 1 5EE8E4DE
 P 5150 3200
@@
 $EndComp
 $Comp
-L Nova-rescue:C-Nova_Microcontroller C?
-U 1 1 5EE97E32
+L Nova-rescue:C-Nova_Microcontroller-Nova-rescue C?
+U 1 1 5F3B6875
 P 9400 3650
 F 0 "C?" H 9515 3696 50  0000 L CNN
@@
 	9400 3800 9400 3950
 $Comp
-L Nova-rescue:C-Nova_Microcontroller C?
+L Nova-rescue:C-Nova_Microcontroller-Nova-rescue C?
 U 1 1 5EE98E46
 P 5450 2350
@@
 	5450 2200 5450 2000
 $Comp
-L Nova-rescue:LED-Nova_Microcontroller D?
+L Nova-rescue:LED-Nova_Microcontroller-Nova-rescue D?
 U 1 1 5EE9CC36
 P 7150 4650
@@
 $EndComp
 $Comp
-L Nova-rescue:R_US-Nova_Microcontroller R?
+L Nova-rescue:R_US-Nova_Microcontroller-Nova-rescue R?
 U 1 1 5EE9D264
 P 6550 4650
@@
 D2+
 $Comp
-L Nova-rescue:R_US-Nova_Microcontroller R?
-U 1 1 5EF2AE69
+L Nova-rescue:R_US-Nova_Microcontroller-Nova-rescue R?
+U 1 1 5F3B687C
 P 6200 3000
 F 0 "R?" V 5995 3000 50  0000 C CNN
@@
 $EndComp
 $Comp
-L Nova-rescue:R_US-Nova_Microcontroller R?
+L Nova-rescue:R_US-Nova_Microcontroller-Nova-rescue R?
 U 1 1 5EF2B785
 P 6450 2750
@@
 $Comp
 L power:PWR_FLAG #FLG?
-U 1 1 5EF372DE
+U 1 1 5F3B687F
 P 8200 2500
 F 0 "#FLG?" H 8200 2575 50  0001 C CNN
@@
 $Comp
 L power:PWR_FLAG #FLG?
-U 1 1 5EF3B232
+U 1 1 5F3B6881
 P 4700 2500
 F 0 "#FLG?" H 4700 2575 50  0001 C CNN

Commit message: Added Gyroscope
Parts:
- C? (x4): symbol Nova-rescue:C-Nova_Microcontroller-Nova-rescue -> Nova-rescue:C-Nova_Microcontroller-Nova-rescue-Nova-rescue
- D?: symbol Nova-rescue:LED-Nova_Microcontroller-Nova-rescue -> Nova-rescue:LED-Nova_Microcontroller-Nova-rescue-Nova-rescue
- F?: symbol Nova-rescue:Fuse-Nova_Microcontroller-Nova-rescue -> Nova-rescue:Fuse-Nova_Microcontroller-Nova-rescue-Nova-rescue
- FB?: symbol Nova-rescue:Ferrite_Bead-Nova_Microcontroller-Nova-rescue -> Nova-rescue:Ferrite_Bead-Nova_Microcontroller-Nova-rescue-Nova-rescue
- J?: symbol Nova-rescue:USB_C_Receptacle-Nova_Microcontroller-Nova-rescue -> Nova-rescue:USB_C_Receptacle-Nova_Microcontroller-Nova-rescue-Nova-rescue
- R? (x5): symbol Nova-rescue:R_US-Nova_Microcontroller-Nova-rescue -> Nova-rescue:R_US-Nova_Microcontroller-Nova-rescue-Nova-rescue
- U?: symbol Nova-rescue:FT234XD-R-Nova_Microcontroller-Nova-rescue -> Nova-rescue:FT234XD-R-Nova_Microcontroller-Nova-rescue-Nova-rescue
Changed lines of the file:
@@
 $Descr A4 11693 8268
 encoding utf-8
-Sheet 4 13
+Sheet 4 14
 Title "Microcontroller"
 Date "2020-07-02"
@@
 $EndBitmap
 $Comp
-L Nova-rescue:USB_C_Receptacle-Nova_Microcontroller-Nova-rescue J?
+L Nova-rescue:USB_C_Receptacle-Nova_Microcontroller-Nova-rescue-Nova-rescue J?
 U 1 1 5EE7E0E1
 P 3900 3500
@@
 Connection ~ 3900 5300
 $Comp
-L Nova-rescue:Fuse-Nova_Microcontroller-Nova-rescue F?
+L Nova-rescue:Fuse-Nova_Microcontroller-Nova-rescue-Nova-rescue F?
 U 1 1 5EE8054D
 P 5050 2500
@@
 	4500 2500 4700 2500
 $Comp
-L Nova-rescue:FT234XD-R-Nova_Microcontroller-Nova-rescue U?
+L Nova-rescue:FT234XD-R-Nova_Microcontroller-Nova-rescue-Nova-rescue U?
 U 1 1 5F3B686B
 P 7900 3500
@@
 $EndComp
 $Comp
-L Nova-rescue:Ferrite_Bead-Nova_Microcontroller-Nova-rescue FB?
+L Nova-rescue:Ferrite_Bead-Nova_Microcontroller-Nova-rescue-Nova-rescue FB?
 U 1 1 5F3B686C
 P 6050 2500
@@
 	6200 2500 8000 2500
 $Comp
-L Nova-rescue:R_US-Nova_Microcontroller-Nova-rescue R?
+L Nova-rescue:R_US-Nova_Microcontroller-Nova-rescue-Nova-rescue R?
 U 1 1 5EE8D72F
 P 5150 3000
@@
 	7250 3600 7500 3600
 $Comp
-L Nova-rescue:C-Nova_Microcontroller-Nova-rescue C?
+L Nova-rescue:C-Nova_Microcontroller-Nova-rescue-Nova-rescue C?
 U 1 1 5F3B6872
 P 5950 3750
@@
 $EndComp
 $Comp
-L Nova-rescue:C-Nova_Microcontroller-Nova-rescue C?
+L Nova-rescue:C-Nova_Microcontroller-Nova-rescue-Nova-rescue C?
 U 1 1 5EE93CEE
 P 6400 3750
@@
 Connection ~ 6200 4050
 $Comp
-L Nova-rescue:R_US-Nova_Microcontroller-Nova-rescue R?
+L Nova-rescue:R_US-Nova_Microcontroller-Nova-rescue-Nova-rescue R?
 U 1 1 5EE8E4DE
 P 5150 3200
@@
 $EndComp
 $Comp
-L Nova-rescue:C-Nova_Microcontroller-Nova-rescue C?
+L Nova-rescue:C-Nova_Microcontroller-Nova-rescue-Nova-rescue C?
 U 1 1 5F3B6875
 P 9400 3650
@@
 	9400 3800 9400 3950
 $Comp
-L Nova-rescue:C-Nova_Microcontroller-Nova-rescue C?
+L Nova-rescue:C-Nova_Microcontroller-Nova-rescue-Nova-rescue C?
 U 1 1 5EE98E46
 P 5450 2350
@@
 	5450 2200 5450 2000
 $Comp
-L Nova-rescue:LED-Nova_Microcontroller-Nova-rescue D?
+L Nova-rescue:LED-Nova_Microcontroller-Nova-rescue-Nova-rescue D?
 U 1 1 5EE9CC36
 P 7150 4650
@@
 $EndComp
 $Comp
-L Nova-rescue:R_US-Nova_Microcontroller-Nova-rescue R?
+L Nova-rescue:R_US-Nova_Microcontroller-Nova-rescue-Nova-rescue R?
 U 1 1 5EE9D264
 P 6550 4650
@@
 D2+
 $Comp
-L Nova-rescue:R_US-Nova_Microcontroller-Nova-rescue R?
+L Nova-rescue:R_US-Nova_Microcontroller-Nova-rescue-Nova-rescue R?
 U 1 1 5F3B687C
 P 6200 3000
@@
 $EndComp
 $Comp
-L Nova-rescue:R_US-Nova_Microcontroller-Nova-rescue R?
+L Nova-rescue:R_US-Nova_Microcontroller-Nova-rescue-Nova-rescue R?
 U 1 1 5EF2B785
 P 6450 2750

Commit message: Added Gyro pins. Organized Schematic
Need to determine if we need the interrupt pins for the sensors.
Parts:
- C? (x4): symbol Nova-rescue:C-Nova_Microcontroller-Nova-rescue-Nova-rescue -> Nova-rescue:C-Nova_Microcontroller-Nova-rescue-Nova-rescue-Nova-rescue
- D?: symbol Nova-rescue:LED-Nova_Microcontroller-Nova-rescue-Nova-rescue -> Nova-rescue:LED-Nova_Microcontroller-Nova-rescue-Nova-rescue-Nova-rescue
- F?: symbol Nova-rescue:Fuse-Nova_Microcontroller-Nova-rescue-Nova-rescue -> Nova-rescue:Fuse-Nova_Microcontroller-Nova-rescue-Nova-rescue-Nova-rescue
- FB?: symbol Nova-rescue:Ferrite_Bead-Nova_Microcontroller-Nova-rescue-Nova-rescue -> Nova-rescue:Ferrite_Bead-Nova_Microcontroller-Nova-rescue-Nova-rescue-Nova-rescue
- J?: symbol Nova-rescue:USB_C_Receptacle-Nova_Microcontroller-Nova-rescue-Nova-rescue -> Nova-rescue:USB_C_Receptacle-Nova_Microcontroller-Nova-rescue-Nova-rescue-Nova-rescue
- R? (x5): symbol Nova-rescue:R_US-Nova_Microcontroller-Nova-rescue-Nova-rescue -> Nova-rescue:R_US-Nova_Microcontroller-Nova-rescue-Nova-rescue-Nova-rescue
- U?: symbol Nova-rescue:FT234XD-R-Nova_Microcontroller-Nova-rescue-Nova-rescue -> Nova-rescue:FT234XD-R-Nova_Microcontroller-Nova-rescue-Nova-rescue-Nova-rescue
Changed lines of the file:
@@
 $EndBitmap
 $Comp
-L Nova-rescue:USB_C_Receptacle-Nova_Microcontroller-Nova-rescue-Nova-rescue J?
+L Nova-rescue:USB_C_Receptacle-Nova_Microcontroller-Nova-rescue-Nova-rescue-Nova-rescue J?
 U 1 1 5EE7E0E1
 P 3900 3500
@@
 Connection ~ 3900 5300
 $Comp
-L Nova-rescue:Fuse-Nova_Microcontroller-Nova-rescue-Nova-rescue F?
+L Nova-rescue:Fuse-Nova_Microcontroller-Nova-rescue-Nova-rescue-Nova-rescue F?
 U 1 1 5EE8054D
 P 5050 2500
@@
 	4500 2500 4700 2500
 $Comp
-L Nova-rescue:FT234XD-R-Nova_Microcontroller-Nova-rescue-Nova-rescue U?
+L Nova-rescue:FT234XD-R-Nova_Microcontroller-Nova-rescue-Nova-rescue-Nova-rescue U?
 U 1 1 5F3B686B
 P 7900 3500
@@
 $EndComp
 $Comp
-L Nova-rescue:Ferrite_Bead-Nova_Microcontroller-Nova-rescue-Nova-rescue FB?
+L Nova-rescue:Ferrite_Bead-Nova_Microcontroller-Nova-rescue-Nova-rescue-Nova-rescue FB?
 U 1 1 5F3B686C
 P 6050 2500
@@
 	6200 2500 8000 2500
 $Comp
-L Nova-rescue:R_US-Nova_Microcontroller-Nova-rescue-Nova-rescue R?
+L Nova-rescue:R_US-Nova_Microcontroller-Nova-rescue-Nova-rescue-Nova-rescue R?
 U 1 1 5EE8D72F
 P 5150 3000
@@
 	7250 3600 7500 3600
 $Comp
-L Nova-rescue:C-Nova_Microcontroller-Nova-rescue-Nova-rescue C?
+L Nova-rescue:C-Nova_Microcontroller-Nova-rescue-Nova-rescue-Nova-rescue C?
 U 1 1 5F3B6872
 P 5950 3750
@@
 $EndComp
 $Comp
-L Nova-rescue:C-Nova_Microcontroller-Nova-rescue-Nova-rescue C?
+L Nova-rescue:C-Nova_Microcontroller-Nova-rescue-Nova-rescue-Nova-rescue C?
 U 1 1 5EE93CEE
 P 6400 3750
@@
 Connection ~ 6200 4050
 $Comp
-L Nova-rescue:R_US-Nova_Microcontroller-Nova-rescue-Nova-rescue R?
+L Nova-rescue:R_US-Nova_Microcontroller-Nova-rescue-Nova-rescue-Nova-rescue R?
 U 1 1 5EE8E4DE
 P 5150 3200
@@
 $EndComp
 $Comp
-L Nova-rescue:C-Nova_Microcontroller-Nova-rescue-Nova-rescue C?
+L Nova-rescue:C-Nova_Microcontroller-Nova-rescue-Nova-rescue-Nova-rescue C?
 U 1 1 5F3B6875
 P 9400 3650
@@
 	9400 3800 9400 3950
 $Comp
-L Nova-rescue:C-Nova_Microcontroller-Nova-rescue-Nova-rescue C?
+L Nova-rescue:C-Nova_Microcontroller-Nova-rescue-Nova-rescue-Nova-rescue C?
 U 1 1 5EE98E46
 P 5450 2350
@@
 	5450 2200 5450 2000
 $Comp
-L Nova-rescue:LED-Nova_Microcontroller-Nova-rescue-Nova-rescue D?
+L Nova-rescue:LED-Nova_Microcontroller-Nova-rescue-Nova-rescue-Nova-rescue D?
 U 1 1 5EE9CC36
 P 7150 4650
@@
 $EndComp
 $Comp
-L Nova-rescue:R_US-Nova_Microcontroller-Nova-rescue-Nova-rescue R?
+L Nova-rescue:R_US-Nova_Microcontroller-Nova-rescue-Nova-rescue-Nova-rescue R?
 U 1 1 5EE9D264
 P 6550 4650
@@
 D2+
 $Comp
-L Nova-rescue:R_US-Nova_Microcontroller-Nova-rescue-Nova-rescue R?
+L Nova-rescue:R_US-Nova_Microcontroller-Nova-rescue-Nova-rescue-Nova-rescue R?
 U 1 1 5F3B687C
 P 6200 3000
@@
 $EndComp
 $Comp
-L Nova-rescue:R_US-Nova_Microcontroller-Nova-rescue-Nova-rescue R?
+L Nova-rescue:R_US-Nova_Microcontroller-Nova-rescue-Nova-rescue-Nova-rescue R?
 U 1 1 5EF2B785
 P 6450 2750

Commit message: Added Pyro Channels
Parts:
- C? (x4): symbol Nova-rescue:C-Nova_Microcontroller-Nova-rescue-Nova-rescue-Nova-rescue -> Nova-rescue:C-Nova_Microcontroller-Nova-rescue-Nova-rescue-Nova-rescue-Nova-rescue
- D?: symbol Nova-rescue:LED-Nova_Microcontroller-Nova-rescue-Nova-rescue-Nova-rescue -> Nova-rescue:LED-Nova_Microcontroller-Nova-rescue-Nova-rescue-Nova-rescue-Nova-rescue
- F?: symbol Nova-rescue:Fuse-Nova_Microcontroller-Nova-rescue-Nova-rescue-Nova-rescue -> Nova-rescue:Fuse-Nova_Microcontroller-Nova-rescue-Nova-rescue-Nova-rescue-Nova-rescue
- FB?: symbol Nova-rescue:Ferrite_Bead-Nova_Microcontroller-Nova-rescue-Nova-rescue-Nova-rescue -> Nova-rescue:Ferrite_Bead-Nova_Microcontroller-Nova-rescue-Nova-rescue-Nova-rescue-Nova-rescue
- J?: symbol Nova-rescue:USB_C_Receptacle-Nova_Microcontroller-Nova-rescue-Nova-rescue-Nova-rescue -> Nova-rescue:USB_C_Receptacle-Nova_Microcontroller-Nova-rescue-Nova-rescue-Nova-rescue-Nova-rescue
- R? (x5): symbol Nova-rescue:R_US-Nova_Microcontroller-Nova-rescue-Nova-rescue-Nova-rescue -> Nova-rescue:R_US-Nova_Microcontroller-Nova-rescue-Nova-rescue-Nova-rescue-Nova-rescue
- U?: symbol Nova-rescue:FT234XD-R-Nova_Microcontroller-Nova-rescue-Nova-rescue-Nova-rescue -> Nova-rescue:FT234XD-R-Nova_Microcontroller-Nova-rescue-Nova-rescue-Nova-rescue-Nova-rescue
Changed lines of the file:
@@
 $Descr A4 11693 8268
 encoding utf-8
-Sheet 4 14
+Sheet 4 16
 Title "Microcontroller"
 Date "2020-07-02"
@@
 $EndBitmap
 $Comp
-L Nova-rescue:USB_C_Receptacle-Nova_Microcontroller-Nova-rescue-Nova-rescue-Nova-rescue J?
+L Nova-rescue:USB_C_Receptacle-Nova_Microcontroller-Nova-rescue-Nova-rescue-Nova-rescue-Nova-rescue J?
 U 1 1 5EE7E0E1
 P 3900 3500
@@
 Connection ~ 3900 5300
 $Comp
-L Nova-rescue:Fuse-Nova_Microcontroller-Nova-rescue-Nova-rescue-Nova-rescue F?
+L Nova-rescue:Fuse-Nova_Microcontroller-Nova-rescue-Nova-rescue-Nova-rescue-Nova-rescue F?
 U 1 1 5EE8054D
 P 5050 2500
@@
 	4500 2500 4700 2500
 $Comp
-L Nova-rescue:FT234XD-R-Nova_Microcontroller-Nova-rescue-Nova-rescue-Nova-rescue U?
+L Nova-rescue:FT234XD-R-Nova_Microcontroller-Nova-rescue-Nova-rescue-Nova-rescue-Nova-rescue U?
 U 1 1 5F3B686B
 P 7900 3500
@@
 $EndComp
 $Comp
-L Nova-rescue:Ferrite_Bead-Nova_Microcontroller-Nova-rescue-Nova-rescue-Nova-rescue FB?
+L Nova-rescue:Ferrite_Bead-Nova_Microcontroller-Nova-rescue-Nova-rescue-Nova-rescue-Nova-rescue FB?
 U 1 1 5F3B686C
 P 6050 2500
@@
 	6200 2500 8000 2500
 $Comp
-L Nova-rescue:R_US-Nova_Microcontroller-Nova-rescue-Nova-rescue-Nova-rescue R?
+L Nova-rescue:R_US-Nova_Microcontroller-Nova-rescue-Nova-rescue-Nova-rescue-Nova-rescue R?
 U 1 1 5EE8D72F
 P 5150 3000
@@
 	7250 3600 7500 3600
 $Comp
-L Nova-rescue:C-Nova_Microcontroller-Nova-rescue-Nova-rescue-Nova-rescue C?
+L Nova-rescue:C-Nova_Microcontroller-Nova-rescue-Nova-rescue-Nova-rescue-Nova-rescue C?
 U 1 1 5F3B6872
 P 5950 3750
@@
 $EndComp
 $Comp
-L Nova-rescue:C-Nova_Microcontroller-Nova-rescue-Nova-rescue-Nova-rescue C?
+L Nova-rescue:C-Nova_Microcontroller-Nova-rescue-Nova-rescue-Nova-rescue-Nova-rescue C?
 U 1 1 5EE93CEE
 P 6400 3750
@@
 Connection ~ 6200 4050
 $Comp
-L Nova-rescue:R_US-Nova_Microcontroller-Nova-rescue-Nova-rescue-Nova-rescue R?
+L Nova-rescue:R_US-Nova_Microcontroller-Nova-rescue-Nova-rescue-Nova-rescue-Nova-rescue R?
 U 1 1 5EE8E4DE
 P 5150 3200
@@
 $EndComp
 $Comp
-L Nova-rescue:C-Nova_Microcontroller-Nova-rescue-Nova-rescue-Nova-rescue C?
+L Nova-rescue:C-Nova_Microcontroller-Nova-rescue-Nova-rescue-Nova-rescue-Nova-rescue C?
 U 1 1 5F3B6875
 P 9400 3650
@@
 	9400 3800 9400 3950
 $Comp
-L Nova-rescue:C-Nova_Microcontroller-Nova-rescue-Nova-rescue-Nova-rescue C?
+L Nova-rescue:C-Nova_Microcontroller-Nova-rescue-Nova-rescue-Nova-rescue-Nova-rescue C?
 U 1 1 5EE98E46
 P 5450 2350
@@
 	5450 2200 5450 2000
 $Comp
-L Nova-rescue:LED-Nova_Microcontroller-Nova-rescue-Nova-rescue-Nova-rescue D?
+L Nova-rescue:LED-Nova_Microcontroller-Nova-rescue-Nova-rescue-Nova-rescue-Nova-rescue D?
 U 1 1 5EE9CC36
 P 7150 4650
@@
 $EndComp
 $Comp
-L Nova-rescue:R_US-Nova_Microcontroller-Nova-rescue-Nova-rescue-Nova-rescue R?
+L Nova-rescue:R_US-Nova_Microcontroller-Nova-rescue-Nova-rescue-Nova-rescue-Nova-rescue R?
 U 1 1 5EE9D264
 P 6550 4650
@@
 D2+
 $Comp
-L Nova-rescue:R_US-Nova_Microcontroller-Nova-rescue-Nova-rescue-Nova-rescue R?
+L Nova-rescue:R_US-Nova_Microcontroller-Nova-rescue-Nova-rescue-Nova-rescue-Nova-rescue R?
 U 1 1 5F3B687C
 P 6200 3000
@@
 $EndComp
 $Comp
-L Nova-rescue:R_US-Nova_Microcontroller-Nova-rescue-Nova-rescue-Nova-rescue R?
+L Nova-rescue:R_US-Nova_Microcontroller-Nova-rescue-Nova-rescue-Nova-rescue-Nova-rescue R?
 U 1 1 5EF2B785
 P 6450 2750
