File: Electrical/Nova/USB-C.sch (KiCad schematic (older format))
At the start: 14 parts

Commit message: Added LED sheet and pins
Parts:
- C? (x4): symbol Nova-rescue:C-Nova_Microcontroller-Nova-rescue-Nova-rescue-Nova-rescue-Nova-rescue -> Nova-rescue:C-Nova_Microcontroller-Nova-rescue-Nova-rescue-Nova-rescue-Nova-rescue-Nova-rescue
- D?: symbol Nova-rescue:LED-Nova_Microcontroller-Nova-rescue-Nova-rescue-Nova-rescue-Nova-rescue -> Nova-rescue:LED-Nova_Microcontroller-Nova-rescue-Nova-rescue-Nova-rescue-Nova-rescue-Nova-rescue
- F?: symbol Nova-rescue:Fuse-Nova_Microcontroller-Nova-rescue-Nova-rescue-Nova-rescue-Nova-rescue -> Nova-rescue:Fuse-Nova_Microcontroller-Nova-rescue-Nova-rescue-Nova-rescue-Nova-rescue-Nova-rescue
- FB?: symbol Nova-rescue:Ferrite_Bead-Nova_Microcontroller-Nova-rescue-Nova-rescue-Nova-rescue-Nova-rescue -> Nova-rescue:Ferrite_Bead-Nova_Microcontroller-Nova-rescue-Nova-rescue-Nova-rescue-Nova-rescue-Nova-rescue
- J?: symbol Nova-rescue:USB_C_Receptacle-Nova_Microcontroller-Nova-rescue-Nova-rescue-Nova-rescue-Nova-rescue -> Nova-rescue:USB_C_Receptacle-Nova_Microcontroller-Nova-rescue-Nova-rescue-Nova-rescue-Nova-rescue-Nova-rescue
- R? (x5): symbol Nova-rescue:R_US-Nova_Microcontroller-Nova-rescue-Nova-rescue-Nova-rescue-Nova-rescue -> Nova-rescue:R_US-Nova_Microcontroller-Nova-rescue-Nova-rescue-Nova-rescue-Nova-rescue-Nova-rescue
- U?: symbol Nova-rescue:FT234XD-R-Nova_Microcontroller-Nova-rescue-Nova-rescue-Nova-rescue-Nova-rescue -> Nova-rescue:FT234XD-R-Nova_Microcontroller-Nova-rescue-Nova-rescue-Nova-rescue-Nova-rescue-Nova-rescue
Changed lines of the file:
@@
 $Descr A4 11693 8268
 encoding utf-8
-Sheet 4 16
+Sheet 4 18
 Title "Microcontroller"
 Date "2020-07-02"
@@
 $EndBitmap
 $Comp
-L Nova-rescue:USB_C_Receptacle-Nova_Microcontroller-Nova-rescue-Nova-rescue-Nova-rescue-Nova-rescue J?
+L Nova-rescue:USB_C_Receptacle-Nova_Microcontroller-Nova-rescue-Nova-rescue-Nova-rescue-Nova-rescue-Nova-rescue J?
 U 1 1 5EE7E0E1
 P 3900 3500
@@
 Connection ~ 3900 5300
 $Comp
-L Nova-rescue:Fuse-Nova_Microcontroller-Nova-rescue-Nova-rescue-Nova-rescue-Nova-rescue F?
+L Nova-rescue:Fuse-Nova_Microcontroller-Nova-rescue-Nova-rescue-Nova-rescue-Nova-rescue-Nova-rescue F?
 U 1 1 5EE8054D
 P 5050 2500
@@
 	4500 2500 4700 2500
 $Comp
-L Nova-rescue:FT234XD-R-Nova_Microcontroller-Nova-rescue-Nova-rescue-Nova-rescue-Nova-rescue U?
+L Nova-rescue:FT234XD-R-Nova_Microcontroller-Nova-rescue-Nova-rescue-Nova-rescue-Nova-rescue-Nova-rescue U?
 U 1 1 5F3B686B
 P 7900 3500
@@
 $EndComp
 $Comp
-L Nova-rescue:Ferrite_Bead-Nova_Microcontroller-Nova-rescue-Nova-rescue-Nova-rescue-Nova-rescue FB?
+L Nova-rescue:Ferrite_Bead-Nova_Microcontroller-Nova-rescue-Nova-rescue-Nova-rescue-Nova-rescue-Nova-rescue FB?
 U 1 1 5F3B686C
 P 6050 2500
@@
 	6200 2500 8000 2500
 $Comp
-L Nova-rescue:R_US-Nova_Microcontroller-Nova-rescue-Nova-rescue-Nova-rescue-Nova-rescue R?
+L Nova-rescue:R_US-Nova_Microcontroller-Nova-rescue-Nova-rescue-Nova-rescue-Nova-rescue-Nova-rescue R?
 U 1 1 5EE8D72F
 P 5150 3000
@@
 	7250 3600 7500 3600
 $Comp
-L Nova-rescue:C-Nova_Microcontroller-Nova-rescue-Nova-rescue-Nova-rescue-Nova-rescue C?
+L Nova-rescue:C-Nova_Microcontroller-Nova-rescue-Nova-rescue-Nova-rescue-Nova-rescue-Nova-rescue C?
 U 1 1 5F3B6872
 P 5950 3750
@@
 $EndComp
 $Comp
-L Nova-rescue:C-Nova_Microcontroller-Nova-rescue-Nova-rescue-Nova-rescue-Nova-rescue C?
+L Nova-rescue:C-Nova_Microcontroller-Nova-rescue-Nova-rescue-Nova-rescue-Nova-rescue-Nova-rescue C?
 U 1 1 5EE93CEE
 P 6400 3750
@@
 Connection ~ 6200 4050
 $Comp
-L Nova-rescue:R_US-Nova_Microcontroller-Nova-rescue-Nova-rescue-Nova-rescue-Nova-rescue R?
+L Nova-rescue:R_US-Nova_Microcontroller-Nova-rescue-Nova-rescue-Nova-rescue-Nova-rescue-Nova-rescue R?
 U 1 1 5EE8E4DE
 P 5150 3200
@@
 $EndComp
 $Comp
-L Nova-rescue:C-Nova_Microcontroller-Nova-rescue-Nova-rescue-Nova-rescue-Nova-rescue C?
+L Nova-rescue:C-Nova_Microcontroller-Nova-rescue-Nova-rescue-Nova-rescue-Nova-rescue-Nova-rescue C?
 U 1 1 5F3B6875
 P 9400 3650
@@
 	9400 3800 9400 3950
 $Comp
-L Nova-rescue:C-Nova_Microcontroller-Nova-rescue-Nova-rescue-Nova-rescue-Nova-rescue C?
+L Nova-rescue:C-Nova_Microcontroller-Nova-rescue-Nova-rescue-Nova-rescue-Nova-rescue-Nova-rescue C?
 U 1 1 5EE98E46
 P 5450 2350
@@
 	5450 2200 5450 2000
 $Comp
-L Nova-rescue:LED-Nova_Microcontroller-Nova-rescue-Nova-rescue-Nova-rescue-Nova-rescue D?
+L Nova-rescue:LED-Nova_Microcontroller-Nova-rescue-Nova-rescue-Nova-rescue-Nova-rescue-Nova-rescue D?
 U 1 1 5EE9CC36
 P 7150 4650
@@
 $EndComp
 $Comp
-L Nova-rescue:R_US-Nova_Microcontroller-Nova-rescue-Nova-rescue-Nova-rescue-Nova-rescue R?
+L Nova-rescue:R_US-Nova_Microcontroller-Nova-rescue-Nova-rescue-Nova-rescue-Nova-rescue-Nova-rescue R?
 U 1 1 5EE9D264
 P 6550 4650
@@
 D2+
 $Comp
-L Nova-rescue:R_US-Nova_Microcontroller-Nova-rescue-Nova-rescue-Nova-rescue-Nova-rescue R?
+L Nova-rescue:R_US-Nova_Microcontroller-Nova-rescue-Nova-rescue-Nova-rescue-Nova-rescue-Nova-rescue R?
 U 1 1 5F3B687C
 P 6200 3000
@@
 $EndComp
 $Comp
-L Nova-rescue:R_US-Nova_Microcontroller-Nova-rescue-Nova-rescue-Nova-rescue-Nova-rescue R?
+L Nova-rescue:R_US-Nova_Microcontroller-Nova-rescue-Nova-rescue-Nova-rescue-Nova-rescue-Nova-rescue R?
 U 1 1 5EF2B785
 P 6450 2750

Commit message: Minor update
Parts:
- C301, C302, C303, C304: renamed from C?; footprint NOVA MCU (STM):C_0805_2012Metric_Pad1.15x1.40mm_HandSolder -> NOVA MCU (STM):C_0805_2012Metric
- D301: renamed from D?; footprint NOVA MCU (STM):LED_0805_2012Metric_Pad1.15x1.40mm_HandSolder -> NOVA MCU (STM):R_0805_2012Metric
- R301, R302, R303, R304, R305: renamed from R?; footprint NOVA MCU (STM):R_0805_2012Metric_Pad1.15x1.40mm_HandSolder -> NOVA MCU (STM):R_0805_2012Metric
- gave numbers to parts that had none: 4
Connections:
- net +3V3: now also C304.1
- net at F301.1, FB301.2: now also C301.2

Commit message: Added Accelerometer
Parts:
- C301, C302, C303, C304: symbol Nova-rescue:C-Nova_Microcontroller-Nova-rescue-Nova-rescue-Nova-rescue-Nova-rescue-Nova-rescue -> Nova-rescue:C-Nova_Microcontroller-Nova-rescue-Nova-rescue-Nova-rescue-Nova-rescue-Nova-rescue-Nova-rescue
- D301: symbol Nova-rescue:LED-Nova_Microcontroller-Nova-rescue-Nova-rescue-Nova-rescue-Nova-rescue-Nova-rescue -> Nova-rescue:LED-Nova_Microcontroller-Nova-rescue-Nova-rescue-Nova-rescue-Nova-rescue-Nova-rescue-Nova-rescue
- F301: symbol Nova-rescue:Fuse-Nova_Microcontroller-Nova-rescue-Nova-rescue-Nova-rescue-Nova-rescue-Nova-rescue -> Nova-rescue:Fuse-Nova_Microcontroller-Nova-rescue-Nova-rescue-Nova-rescue-Nova-rescue-Nova-rescue-Nova-rescue
- FB301: symbol Nova-rescue:Ferrite_Bead-Nova_Microcontroller-Nova-rescue-Nova-rescue-Nova-rescue-Nova-rescue-Nova-rescue -> Nova-rescue:Ferrite_Bead-Nova_Microcontroller-Nova-rescue-Nova-rescue-Nova-rescue-Nova-rescue-Nova-rescue-Nova-rescue
- J301: symbol Nova-rescue:USB_C_Receptacle-Nova_Microcontroller-Nova-rescue-Nova-rescue-Nova-rescue-Nova-rescue-Nova-rescue -> Nova-rescue:USB_C_Receptacle-Nova_Microcontroller-Nova-rescue-Nova-rescue-Nova-rescue-Nova-rescue-Nova-rescue-Nova-resc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
- R301, R302, R303, R304, R305: symbol Nova-rescue:R_US-Nova_Microcontroller-Nova-rescue-Nova-rescue-Nova-rescue-Nova-rescue-Nova-rescue -> Nova-rescue:R_US-Nova_Microcontroller-Nova-rescue-Nova-rescue-Nova-rescue-Nova-rescue-Nova-rescue-Nova-rescue
- U301: symbol Nova-rescue:FT234XD-R-Nova_Microcontroller-Nova-rescue-Nova-rescue-Nova-rescue-Nova-rescue-Nova-rescue -> Nova-rescue:FT234XD-R-Nova_Microcontroller-Nova-rescue-Nova-rescue-Nova-rescue-Nova-rescue-Nova-rescue-Nova-rescue
Changed lines of the file:
@@
 $Descr A4 11693 8268
 encoding utf-8
-Sheet 3 18
+Sheet 3 19
 Title "Microcontroller"
 Date "2020-07-02"
@@
 $EndBitmap
 $Comp
-L Nova-rescue:USB_C_Receptacle-Nova_Microcontroller-Nova-rescue-Nova-rescue-Nova-rescue-Nova-rescue-Nova-rescue J301
+L Nova-rescue:USB_C_Receptacle-Nova_Microcontroller-Nova-rescue-Nova-rescue-Nova-rescue-Nova-rescue-Nova-rescue-Nova-rescue J301
 U 1 1 5EE7E0E1
 P 3900 3500
@@
 Connection ~ 3900 5300
 $Comp
-L Nova-rescue:Fuse-Nova_Microcontroller-Nova-rescue-Nova-rescue-Nova-rescue-Nova-rescue-Nova-rescue F301
+L Nova-rescue:Fuse-Nova_Microcontroller-Nova-rescue-Nova-rescue-Nova-rescue-Nova-rescue-Nova-rescue-Nova-rescue F301
 U 1 1 5EE8054D
 P 5050 2500
@@
 	4500 2500 4700 2500
 $Comp
-L Nova-rescue:FT234XD-R-Nova_Microcontroller-Nova-rescue-Nova-rescue-Nova-rescue-Nova-rescue-Nova-rescue U301
+L Nova-rescue:FT234XD-R-Nova_Microcontroller-Nova-rescue-Nova-rescue-Nova-rescue-Nova-rescue-Nova-rescue-Nova-rescue U301
 U 1 1 5F3B686B
 P 7900 3500
@@
 $EndComp
 $Comp
-L Nova-rescue:Ferrite_Bead-Nova_Microcontroller-Nova-rescue-Nova-rescue-Nova-rescue-Nova-rescue-Nova-rescue FB301
+L Nova-rescue:Ferrite_Bead-Nova_Microcontroller-Nova-rescue-Nova-rescue-Nova-rescue-Nova-rescue-Nova-rescue-Nova-rescue FB301
 U 1 1 5F3B686C
 P 6050 2500
@@
 	6200 2500 8000 2500
 $Comp
-L Nova-rescue:R_US-Nova_Microcontroller-Nova-rescue-Nova-rescue-Nova-rescue-Nova-rescue-Nova-rescue R301
+L Nova-rescue:R_US-Nova_Microcontroller-Nova-rescue-Nova-rescue-Nova-rescue-Nova-rescue-Nova-rescue-Nova-rescue R301
 U 1 1 5EE8D72F
 P 5150 3000
@@
 	7250 3600 7500 3600
 $Comp
-L Nova-rescue:C-Nova_Microcontroller-Nova-rescue-Nova-rescue-Nova-rescue-Nova-rescue-Nova-rescue C302
+L Nova-rescue:C-Nova_Microcontroller-Nova-rescue-Nova-rescue-Nova-rescue-Nova-rescue-Nova-rescue-Nova-rescue C302
 U 1 1 5F3B6872
 P 5950 3750
@@
 $EndComp
 $Comp
-L Nova-rescue:C-Nova_Microcontroller-Nova-rescue-Nova-rescue-Nova-rescue-Nova-rescue-Nova-rescue C303
+L Nova-rescue:C-Nova_Microcontroller-Nova-rescue-Nova-rescue-Nova-rescue-Nova-rescue-Nova-rescue-Nova-rescue C303
 U 1 1 5EE93CEE
 P 6400 3750
@@
 Connection ~ 6200 4050
 $Comp
-L Nova-rescue:R_US-Nova_Microcontroller-Nova-rescue-Nova-rescue-Nova-rescue-Nova-rescue-Nova-rescue R302
+L Nova-rescue:R_US-Nova_Microcontroller-Nova-rescue-Nova-rescue-Nova-rescue-Nova-rescue-Nova-rescue-Nova-rescue R302
 U 1 1 5EE8E4DE
 P 5150 3200
@@
 $EndComp
 $Comp
-L Nova-rescue:C-Nova_Microcontroller-Nova-rescue-Nova-rescue-Nova-rescue-Nova-rescue-Nova-rescue C304
+L Nova-rescue:C-Nova_Microcontroller-Nova-rescue-Nova-rescue-Nova-rescue-Nova-rescue-Nova-rescue-Nova-rescue C304
 U 1 1 5F3B6875
 P 9400 3650
@@
 	9400 3800 9400 3950
 $Comp
-L Nova-rescue:C-Nova_Microcontroller-Nova-rescue-Nova-rescue-Nova-rescue-Nova-rescue-Nova-rescue C301
+L Nova-rescue:C-Nova_Microcontroller-Nova-rescue-Nova-rescue-Nova-rescue-Nova-rescue-Nova-rescue-Nova-rescue C301
 U 1 1 5EE98E46
 P 5450 2350
@@
 	5450 2200 5450 2000
 $Comp
-L Nova-rescue:LED-Nova_Microcontroller-Nova-rescue-Nova-rescue-Nova-rescue-Nova-rescue-Nova-rescue D301
+L Nova-rescue:LED-Nova_Microcontroller-Nova-rescue-Nova-rescue-Nova-rescue-Nova-rescue-Nova-rescue-Nova-rescue D301
 U 1 1 5EE9CC36
 P 7150 4650
@@
 $EndComp
 $Comp
-L Nova-rescue:R_US-Nova_Microcontroller-Nova-rescue-Nova-rescue-Nova-rescue-Nova-rescue-Nova-rescue R305
+L Nova-rescue:R_US-Nova_Microcontroller-Nova-rescue-Nova-rescue-Nova-rescue-Nova-rescue-Nova-rescue-Nova-rescue R305
 U 1 1 5EE9D264
 P 6550 4650
@@
 D2+
 $Comp
-L Nova-rescue:R_US-Nova_Microcontroller-Nova-rescue-Nova-rescue-Nova-rescue-Nova-rescue-Nova-rescue R303
+L Nova-rescue:R_US-Nova_Microcontroller-Nova-rescue-Nova-rescue-Nova-rescue-Nova-rescue-Nova-rescue-Nova-rescue R303
 U 1 1 5F3B687C
 P 6200 3000
@@
 $EndComp
 $Comp
-L Nova-rescue:R_US-Nova_Microcontroller-Nova-rescue-Nova-rescue-Nova-rescue-Nova-rescue-Nova-rescue R304
+L Nova-rescue:R_US-Nova_Microcontroller-Nova-rescue-Nova-rescue-Nova-rescue-Nova-rescue-Nova-rescue-Nova-rescue R304
 U 1 1 5EF2B785
 P 6450 2750
