File: Electrical/Nova/LED Indication.sch (KiCad schematic (older format))
At the start: 0 parts

Commit message: Added LED sheet and pins
Parts:
- added D?: ASMB-MTB0-0A3A2, LED_SMD:LED_Avago_PLCC4_3.2x2.8mm_CW, symbol LED:ASMB-MTB0-0A3A2
- added R? (x3): 330, symbol Device:R_US
Connections:
- new net: D?.2 (BK), R?.1
- new net: D?.3 (GK), R?.1
- new net: D?.4 (RK), R?.1
- new net +3V3: D?.1 (A)
- new net LED_BLUE: R?.2
- new net LED_GREEN: R?.2
- new net LED_RED: R?.2
Changed lines of the file:
@@
 $Descr A4 11693 8268
 encoding utf-8
-Sheet 2 16
+Sheet 2 18
 Title ""
 Date ""
@@
 Comment4 ""
 $EndDescr
+$Comp
+L LED:ASMB-MTB0-0A3A2 D?
+U 1 1 5F47D6CA
+P 6250 3550
+F 0 "D?" H 6250 4067 50  0000 C CNN
+F 1 "ASMB-MTB0-0A3A2" H 6250 3976 50  0000 C CNN
+F 2 "LED_SMD:LED_Avago_PLCC4_3.2x2.8mm_CW" H 6250 4050 50  0001 C CNN
+F 3 "https://docs.broadcom.com/docs/AV02-4186EN" H 6250 3100 50  0001 C CNN
+	1    6250 3550
+	1    0    0    -1
+$EndComp
+$Comp
+L Device:R_US R?
+U 1 1 5F47E7A4
+P 5250 3350
+F 0 "R?" V 5045 3350 50  0000 C CNN
+F 1 "330" V 5136 3350 50  0000 C CNN
+F 2 "" V 5290 3340 50  0001 C CNN
+F 3 "~" H 5250 3350 50  0001 C CNN
+	1    5250 3350
+	0    1    1    0
+$EndComp
+$Comp
+L Device:R_US R?
+U 1 1 5F47EC03
+P 4950 3550
+F 0 "R?" V 4745 3550 50  0000 C CNN
+F 1 "330" V 4836 3550 50  0000 C CNN
+F 2 "" V 4990 3540 50  0001 C CNN
+F 3 "~" H 4950 3550 50  0001 C CNN
+	1    4950 3550
+	0    1    1    0
+$EndComp
+$Comp
+L Device:R_US R?
+U 1 1 5F47F1A5
+P 5250 3750
+F 0 "R?" V 5450 3750 50  0000 C CNN
+F 1 "330" V 5350 3750 50  0000 C CNN
+F 2 "" V 5290 3740 50  0001 C CNN
+F 3 "~" H 5250 3750 50  0001 C CNN
+	1    5250 3750
+	0    1    1    0
+$EndComp
+Wire Wire Line
+	6050 3350 5400 3350
+Wire Wire Line
+	5100 3550 6050 3550
+Wire Wire Line
+	6050 3750 5400 3750
+$Comp
+L power:+3.3V #PWR?
+U 1 1 5F47FF39
+P 6950 3550
+F 0 "#PWR?" H 6950 3400 50  0001 C CNN
+F 1 "+3.3V" V 6965 3678 50  0000 L CNN
+F 2 "" H 6950 3550 50  0001 C CNN
+F 3 "" H 6950 3550 50  0001 C CNN
+	1    6950 3550
+	0    1    1    0
+$EndComp
+Wire Wire Line
+	6450 3550 6950 3550
+Text HLabel 4500 3350 0    79   Input ~ 0
+LED_RED
+Text HLabel 4500 3750 0    79   Input ~ 0
+LED_BLUE
+Text HLabel 4500 3550 0    79   Input ~ 0
+LED_GREEN
+Wire Wire Line
+	4500 3350 5100 3350
+Wire Wire Line
+	4500 3550 4800 3550
+Wire Wire Line
+	4500 3750 5100 3750
 $EndSCHEMATC

Commit message: Minor update
Parts:
- R201, R202, R203: renamed from R?; footprint (none) -> NOVA MCU (STM):R_0805_2012Metric
- gave numbers to parts that had none: 1
Changed lines of the file:
@@
 $EndDescr
 $Comp
-L LED:ASMB-MTB0-0A3A2 D?
+L LED:ASMB-MTB0-0A3A2 D201
 U 1 1 5F47D6CA
 P 6250 3550
-F 0 "D?" H 6250 4067 50  0000 C CNN
+F 0 "D201" H 6250 4067 50  0000 C CNN
 F 1 "ASMB-MTB0-0A3A2" H 6250 3976 50  0000 C CNN
 F 2 "LED_SMD:LED_Avago_PLCC4_3.2x2.8mm_CW" H 6250 4050 50  0001 C CNN
@@
 $EndComp
 $Comp
-L Device:R_US R?
+L Device:R_US R202
 U 1 1 5F47E7A4
 P 5250 3350
-F 0 "R?" V 5045 3350 50  0000 C CNN
+F 0 "R202" V 5045 3350 50  0000 C CNN
 F 1 "330" V 5136 3350 50  0000 C CNN
-F 2 "" V 5290 3340 50  0001 C CNN
+F 2 "NOVA MCU (STM):R_0805_2012Metric" V 5290 3340 50  0001 C CNN
 F 3 "~" H 5250 3350 50  0001 C CNN
 	1    5250 3350
@@
 $EndComp
 $Comp
-L Device:R_US R?
+L Device:R_US R201
 U 1 1 5F47EC03
 P 4950 3550
-F 0 "R?" V 4745 3550 50  0000 C CNN
+F 0 "R201" V 4745 3550 50  0000 C CNN
 F 1 "330" V 4836 3550 50  0000 C CNN
-F 2 "" V 4990 3540 50  0001 C CNN
+F 2 "NOVA MCU (STM):R_0805_2012Metric" V 4990 3540 50  0001 C CNN
 F 3 "~" H 4950 3550 50  0001 C CNN
 	1    4950 3550
@@
 $EndComp
 $Comp
-L Device:R_US R?
+L Device:R_US R203
 U 1 1 5F47F1A5
 P 5250 3750
-F 0 "R?" V 5450 3750 50  0000 C CNN
+F 0 "R203" V 5450 3750 50  0000 C CNN
 F 1 "330" V 5350 3750 50  0000 C CNN
-F 2 "" V 5290 3740 50  0001 C CNN
+F 2 "NOVA MCU (STM):R_0805_2012Metric" V 5290 3740 50  0001 C CNN
 F 3 "~" H 5250 3750 50  0001 C CNN
 	1    5250 3750
@@
 	6050 3750 5400 3750
 $Comp
-L power:+3.3V #PWR?
+L power:+3.3V #PWR0201
 U 1 1 5F47FF39
 P 6950 3550
-F 0 "#PWR?" H 6950 3400 50  0001 C CNN
+F 0 "#PWR0201" H 6950 3400 50  0001 C CNN
 F 1 "+3.3V" V 6965 3678 50  0000 L CNN
 F 2 "" H 6950 3550 50  0001 C CNN

Commit message: Switched All Capacitors and Resistors to 0603
Parts:
- R201, R202, R203: footprint NOVA MCU (STM):R_0805_2012Metric -> NOVA MCU (STM):R_0603_1608Metric
Changed lines of the file:
@@
 F 0 "R202" V 5045 3350 50  0000 C CNN
 F 1 "330" V 5136 3350 50  0000 C CNN
-F 2 "NOVA MCU (STM):R_0805_2012Metric" V 5290 3340 50  0001 C CNN
+F 2 "NOVA MCU (STM):R_0603_1608Metric" V 5290 3340 50  0001 C CNN
 F 3 "~" H 5250 3350 50  0001 C CNN
 	1    5250 3350
@@
 F 0 "R201" V 4745 3550 50  0000 C CNN
 F 1 "330" V 4836 3550 50  0000 C CNN
-F 2 "NOVA MCU (STM):R_0805_2012Metric" V 4990 3540 50  0001 C CNN
+F 2 "NOVA MCU (STM):R_0603_1608Metric" V 4990 3540 50  0001 C CNN
 F 3 "~" H 4950 3550 50  0001 C CNN
 	1    4950 3550
@@
 F 0 "R203" V 5450 3750 50  0000 C CNN
 F 1 "330" V 5350 3750 50  0000 C CNN
-F 2 "NOVA MCU (STM):R_0805_2012Metric" V 5290 3740 50  0001 C CNN
+F 2 "NOVA MCU (STM):R_0603_1608Metric" V 5290 3740 50  0001 C CNN
 F 3 "~" H 5250 3750 50  0001 C CNN
 	1    5250 3750
