File: Electrical/Nova/Nova.kicad_pcb (KiCad board)
At the start: 4 copper layers, 36.5 x 94.1 mm, 89 parts

Commit message: Electrical REV1
Parts:
- removed G***: LOGO, logo:Logo
- 3v3Reg1, C1, C10, C11, C14, C15, C16, C17, C18, C19, C2, C20, C21, C24, C25, C26, C3, C5, C6, C7, C8, C9, D1, D3, D4, F1, FB1, H1, H2, H3, H4, IC1, J1, J2, J3, J4, J5, LS1, Q1, Q2, Q3, Q4, Q5, Q6, Q7, R11, R12, R13, R15, R16, R17, R18, R6, R7, R8, R9, S1, U1, U2, U4, U5, USB1, Y1, Y2, xt1: renamed from  
- Barometer1: renamed from  ; value (none) -> MS560702BA03-50
- C13: renamed from C 
- C22: renamed from  ; value 10uf -> 10uF
- C23: renamed from  ; value 0.1uf -> 100nF
- C27: renamed from  ; value 0.33 uF -> 0.33uF
- C28: renamed from  ; value 0.1 uF -> 100nF
- C29, C30, C31: renamed from  ; footprint Capacitor_SMD:C_0603_1608Metric -> Capacitor_SMD:C_0603_1608Metric_Pad1.05x0.95mm_HandSolder
- C4: renamed from  ; value 0.1uF -> 100nF
- R1, R2, R21, R22, R23, R24, R3, R5: renamed from  ; footprint Resistor_SMD:R_0603_1608Metric -> Resistor_SMD:R_0603_1608Metric_Pad1.05x0.95mm_HandSolder
- R10, R14: renamed from  ; value (none) -> 10k
- R4: renamed from  ; value TBD -> 10k
- U3: renamed from  ; footprint FHSD:W25N512GVPIT -> FHSD:SON127P800X600X80-9N
- moved S1 1.95 mm to (138.1, 62.6)
- moved C26 0.41 mm to (160.2, 66.7), turned to 180 degrees
- moved U3 0.15 mm to (161.7, 68.1)
Connections:
- IC1 pad 2: (no net) -> GND
- U1 pad 34: (no net) -> /FLASH_CS
- U3 pad 1: (no net) -> /FLASH_CS
- U3 pad 2: /MISO -> /H_MISO
- U3 pad 5: /MOSI -> /H_MOSI
- U3 pad 6: /SCLK -> /H_SCLK
Routing:
- net /SCLK: track 72.6 -> 35.7 mm
- net /MOSI: track 67.1 -> 36.0 mm, vias 6 -> 5
- net /H_MOSI: track 17.5 -> 42.1 mm, vias 0 -> 2
- net /MISO: track 63.7 -> 40.5 mm
- net /H_SCLK: track 24.6 -> 42.1 mm, vias 1 -> 2
- net /H_MISO: track 18.7 -> 34.0 mm, vias 1 -> 3
- net /FLASH_CS: track 0.00 -> 6.28 mm
- net GND: track 165.9 -> 170.2 mm, vias 40 -> 41
- net /RESET: track 38.4 -> 41.0 mm
- net +3V3: track 90.4 -> 91.1 mm
- added copper zone on B.Cu, net GND
- added copper zone on F.Cu, net GND

Commit message: Semi-Final Changes to REV1.0 Board
Parts:
- 3v3 REG: renamed from 3v3Reg1
- BATT POWER: renamed from xt1
- Barometer1: value MS560702BA03-50 -> B
- Battery Monitor: renamed from U5
- PYRO 1: renamed from J3
- PYRO 2: renamed from J2
- PYRO 3: renamed from J4
- renumbered U2 to A, LS1 to BUZZER, U3 to FLASH, U4 to FTDI, IC1 to G, U1 to STM32F401RBT, USB1 to USB-C
Routing:
- net /LED_BLUE: track 12.7 -> 13.3 mm
Other:
- net class Default: clearance 0.2 -> 0.15
- rule trace_clearance: 0.2 -> 0.15
- board text added: "NOVA REV 1.0"
- board text removed: "BOTTOM"

Commit message: Added Logo to Rev 1.0
Parts:
- added G***: LOGO, Rev1Logo:Logo3, B.Cu at (155.6, 89.3)

Commit message: Removed Obsolete Components & Modified Format  and Misc
Parts:
- removed 3v3 REG: AZ1117EH-3.3TRG1, Power:SOT230P700X180-4N
- removed A: H3LIS331DL, Accelerometer_Breakout:TFLGA-16_3x3mm
- removed BATT POWER: Conn_01x02, Connector_AMASS:AMASS_XT30PW-M_1x02_P2.50mm_Horizontal
- removed BUZZER: PS1440P02BT, Transducer:BUZZER_PS1440P02BT
- removed Barometer1: B, Barometer:MS560702BA03-50
- removed Battery Monitor: OP179GRT, Package_TO_SOT_SMD:SOT-23-5
- removed C1, C10, C14, C16, C2, C23, C25, C26, C28, C29, C3, C4, C5, C6, C7, C8, C9: 100nF, Capacitor_SMD:C_0603_1608Metric_Pad1.05x0.95mm_HandSolder
- removed C11, C13, C30: 4.7uF, Capacitor_SMD:C_0603_1608Metric_Pad1.05x0.95mm_HandSolder
- removed C15, C17: 1uF, Capacitor_SMD:C_0603_1608Metric_Pad1.05x0.95mm_HandSolder
- removed C18, C21: 18pf, Capacitor_SMD:C_0603_1608Metric_Pad1.05x0.95mm_HandSolder
- removed C19, C20: 10pf, Capacitor_SMD:C_0603_1608Metric_Pad1.05x0.95mm_HandSolder
- removed C22: 10uF, Capacitor_SMD:C_0603_1608Metric_Pad1.05x0.95mm_HandSolder
- removed C24: 1mF, PyroChannel:CP_Radial_D10.0mm_P5.00mm
- removed C27: 0.33uF, Capacitor_SMD:C_0603_1608Metric_Pad1.05x0.95mm_HandSolder
- removed C31: 10nF, Capacitor_SMD:C_0603_1608Metric_Pad1.05x0.95mm_HandSolder
- removed D1: ASMB-MTB0-0A3A2, LED_SMD:LED_Avago_PLCC4_3.2x2.8mm_CW
- removed D3, D4: DIODE, Diode_SMD:D_0805_2012Metric_Pad1.15x1.40mm_HandSolder
- removed F1: 500mA, Fuse:Fuse_1206_3216Metric_Pad1.42x1.75mm_HandSolder
- removed FB1: 600 OHM, Resistor_SMD:R_0805_2012Metric_Pad1.15x1.40mm_HandSolder
- removed FLASH: W25N512GVPIT, FHSD:SON127P800X600X80-9N
- removed FTDI: FT232RL-REEL, Footrpint Library:SOP65P780X200-28N
- removed G: BMI088, Gyroscope:16-LGA-(4.5x3)
- removed G***: LOGO, Rev1Logo:Logo3
- removed H1, H2, H3, H4: MountingHole, MountingHole:MountingHole_3mm
- removed J1: Conn_01x06_Male, NOVA MCU (STM):j-link_6_pin_needle
- removed J5: Conn_02x10_Counter_Clockwise, Connector_PinSocket_2.54mm:PinSocket_2x10_P2.54mm_Vertical
- removed Micro_SD1: Micro_SD_Card, Connector_Card:microSD_HC_Wuerth_693072010801
- removed PYRO 1: Conn_01x02_Female, PyroChannel:2_pin_screw_terminal
- removed PYRO 2: Conn_01x02_Female, PyroChannel:2_pin_screw_terminal
- removed PYRO 3: Conn_01x02_Female, PyroChannel:2_pin_screw_terminal
- removed Q1, Q2, Q3, Q4, Q5, Q6, Q7: IRLML6344TRPBFee, PyroChannel:SOT-23
- removed R1, R2, R3: 330, Resistor_SMD:R_0603_1608Metric_Pad1.05x0.95mm_HandSolder
- removed R10, R11, R13, R14, R15, R17, R18, R4, R5, R6, R7, R9: 10k, Resistor_SMD:R_0603_1608Metric_Pad1.05x0.95mm_HandSolder
- removed R12, R16, R8: 3.3, PyroChannel:TO-263-2_TabPin1
- removed R21, R22: 5k, Resistor_SMD:R_0603_1608Metric_Pad1.05x0.95mm_HandSolder
- removed R23: 95.5k, Resistor_SMD:R_0603_1608Metric_Pad1.05x0.95mm_HandSolder
- removed R24: 47k, Resistor_SMD:R_0603_1608Metric_Pad1.05x0.95mm_HandSolder
- removed S1: KSR223GLFG, NOVA MCU (STM):KSR223GLFG
- removed STM32F401RBT: STM32F401RBTx, NOVA MCU (STM):LQFP-64_10x10mm_P0.5mm
- removed USB-C: USB_C_Receptacle, Connector_USB:USB_C_Receptacle_Amphenol_12401610E4-2A
- removed Y1: ECS-260-8-36B-CKY-TR, NOVA MCU (STM):ECX-2236B
- removed Y2: JTX310, NOVA MCU (STM):JTX310
Routing:
- net GND: track 170.2 -> 0.00 mm, vias 41 -> 0
- net +BATT: track 111.7 -> 0.00 mm, vias 2 -> 0
- net +3V3: track 91.2 -> 0.00 mm, vias 24 -> 0
- net /CONTINUITY1: track 86.9 -> 0.00 mm, vias 3 -> 0
- net /FIRE1: track 84.0 -> 0.00 mm, vias 3 -> 0
- net /CONTINUITY2: track 82.7 -> 0.00 mm, vias 3 -> 0
- net /CONTINUITY3: track 75.5 -> 0.00 mm, vias 3 -> 0
- net /FIRE2: track 75.1 -> 0.00 mm, vias 3 -> 0
- net /FIRE3: track 71.9 -> 0.00 mm, vias 3 -> 0
- net /ARM: track 68.0 -> 0.00 mm, vias 2 -> 0
- net /SD_CS: track 64.9 -> 0.00 mm, vias 1 -> 0
- net /TXD: track 62.7 -> 0.00 mm, vias 2 -> 0
- net /RXD: track 55.2 -> 0.00 mm, vias 2 -> 0
- net /ACCELEROMETER_CS: track 50.5 -> 0.00 mm, vias 2 -> 0
- net /GYRO_CS: track 44.4 -> 0.00 mm, vias 2 -> 0
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- removed copper zone on 3.3V, net +3V3
- removed copper zone on B.Cu, net GND
- removed copper zone on F.Cu, net GND
- removed copper zone on GND, net GND
Other:
- board outline removed
- board text removed: "NOVA REV 1.0"
- board text removed: "TOP"

Commit message: Finished adding footprints
Parts:
- added 3v3Reg1: AZ1117EH-3.3TRG1, Power:SOT230P700X180-4N, F.Cu at (155.8, 70.9)
- added BZ1: Buzzer, Transducer:XDCR_CMT-7525-80-SMT-TR, F.Cu at (93.7, 124.8)
- added C1: 0.33uF, Capacitor_SMD:C_0402_1005Metric, F.Cu at (152.1, 79.1)
- added C10: 100nF, Capacitor_SMD:C_0402_1005Metric, F.Cu at (178.6, 119.0)
- added C11: 4.7uF, Capacitor_SMD:C_0402_1005Metric, F.Cu at (181.5, 121.0)
- added C12: 100nF, Capacitor_SMD:C_0402_1005Metric, F.Cu at (189.5, 89.0)
- added C13: 4.7uF, Capacitor_SMD:C_0402_1005Metric, F.Cu at (178.6, 123.0)
- added C14: 100nF, Capacitor_SMD:C_0402_1005Metric, F.Cu at (181.5, 119.0)
- added C15: 1uF, Capacitor_SMD:C_0402_1005Metric, F.Cu at (178.6, 121.0)
- added C16: 100nF, Capacitor_SMD:C_0402_1005Metric, F.Cu at (192.4, 87.0)
- added C17: 100nF, Capacitor_SMD:C_0402_1005Metric, F.Cu at (189.5, 91.0)
- added C18: 18pf, Capacitor_SMD:C_0402_1005Metric, F.Cu at (170.5, 119.4)
- added C19: 10pf, Capacitor_SMD:C_0402_1005Metric, F.Cu at (170.5, 117.4)
- added C2: 100nF, Capacitor_SMD:C_0402_1005Metric, F.Cu at (156.9, 76.0)
- added C20: 10pf, Capacitor_SMD:C_0402_1005Metric, F.Cu at (171.1, 115.4)
- added C21: 18pf, Capacitor_SMD:C_0402_1005Metric, F.Cu at (167.5, 118.2)
- added C22: 10uF, Capacitor_SMD:C_0402_1005Metric, F.Cu at (197.8, 110.7)
- added C23: 100nF, Capacitor_SMD:C_0402_1005Metric, F.Cu at (197.8, 108.7)
- added C24: 1mF, PyroChannel:CP_Radial_D10.0mm_P5.00mm, F.Cu at (115.9, 72.6)
- added C25: 100nF, Capacitor_SMD:C_0402_1005Metric, F.Cu at (151.3, 95.2)
- added C26: 100nF, Capacitor_SMD:C_0402_1005Metric, F.Cu at (178.2, 88.5)
- added C27: 10uF, Capacitor_SMD:C_0402_1005Metric, F.Cu at (192.4, 89.0)
- added C29: 100nF, Capacitor_SMD:C_0402_1005Metric, F.Cu at (150.8, 126.8)
- added C3: 100nF, Capacitor_SMD:C_0402_1005Metric, F.Cu at (173.2, 99.2)
- added C30: 4.7uF, Capacitor_SMD:C_0402_1005Metric, F.Cu at (155.4, 119.4)
- added C31: 10nF, Capacitor_SMD:C_0402_1005Metric, F.Cu at (147.9, 126.8)
- added C5: 10nF, Capacitor_SMD:C_0402_1005Metric, F.Cu at (189.5, 87.0)
- added C6: 100nF, Capacitor_SMD:C_0402_1005Metric, F.Cu at (187.3, 119.0)
- added C7: 100nF, Capacitor_SMD:C_0402_1005Metric, F.Cu at (184.4, 121.0)
- added C8: 100nF, Capacitor_SMD:C_0402_1005Metric, F.Cu at (181.5, 123.0)
- added C9: 100nF, Capacitor_SMD:C_0402_1005Metric, F.Cu at (184.4, 119.0)
- added D1: ASMB-MTB0-0A3A2, LED_SMD:LED_Avago_PLCC4_3.2x2.8mm_CW, F.Cu at (113.4, 122.3)
- added D2: DIODE, Diode_SMD:D_0805_2012Metric_Pad1.15x1.40mm_HandSolder, F.Cu at (100.8, 121.6)
- added D3: DIODE, Diode_SMD:D_0805_2012Metric_Pad1.15x1.40mm_HandSolder, F.Cu at (153.1, 76.5)
- added D4: DIODE, Diode_SMD:D_0805_2012Metric_Pad1.15x1.40mm_HandSolder, F.Cu at (163.0, 68.3)
- added D5: LED, LED_SMD:LED_0402_1005Metric, F.Cu at (145.0, 126.8)
- added D6: LED, LED_SMD:LED_0402_1005Metric, F.Cu at (155.7, 115.4)
- added F1: 500mA, Fuse:Fuse_1206_3216Metric_Pad1.42x1.75mm_HandSolder, F.Cu at (135.6, 127.3)
- added FB1: 600 OHM, Resistor_SMD:R_0805_2012Metric_Pad1.15x1.40mm_HandSolder, F.Cu at (141.0, 127.3)
- added H1: MountingHole, MountingHole:MountingHole_3mm, F.Cu at (114.3, 105.5)
- added H2: MountingHole, MountingHole:MountingHole_3mm, F.Cu at (121.8, 98.0)
- added H3: MountingHole, MountingHole:MountingHole_3mm, F.Cu at (105.2, 112.4)
- added H4: MountingHole, MountingHole:MountingHole_3mm, F.Cu at (114.3, 98.0)
- added J1: Conn_01x05_Male_Programmer, Connector_PinHeader_2.54mm:PinHeader_1x05_P2.54mm_Vertical, F.Cu at (172.1, 69.1)
- added J2: Conn_MX_530480710, Connector_Molex:Molex_PicoBlade_53048-0710_1x07_P1.25mm_Horizontal, F.Cu at (91.4, 111.0)
- added J3: Conn_02x05_Counter_Clockwise, Connector_PinSocket_2.54mm:PinSocket_2x05_P2.54mm_Vertical, F.Cu at (93.8, 96.5)
- added J4: Conn_01x02_Female, TerminalBlock_Phoenix:TerminalBlock_Phoenix_PTSM-0,5-2-2.5-H-THR_1x02_P2.50mm_Horizontal, F.Cu at (106.5, 75.0)
- added J5: Conn_01x04_Female, TerminalBlock_Phoenix:TerminalBlock_Phoenix_PTSM-0,5-4-2.5-H-THR_1x04_P2.50mm_Horizontal, F.Cu at (92.3, 87.1)
- added J6: Conn_01x04_Female, TerminalBlock_Phoenix:TerminalBlock_Phoenix_PTSM-0,5-4-2.5-H-THR_1x04_P2.50mm_Horizontal, F.Cu at (92.3, 75.0)
- added Micro_SD1: WE_693072010801, Connector_Card:microSD_HC_Wuerth_693072010801, F.Cu at (141.2, 102.0)
- added Q1: IRLML6344TRPBFee, PyroChannel:SOT-23, F.Cu at (194.0, 117.7)
- added Q10: MMBF4393, Package_TO_SOT_SMD:SOT-23, F.Cu at (100.6, 125.4)
- added Q2: IRLML6344TRPBFee, PyroChannel:SOT-23, F.Cu at (183.8, 110.7)
- added Q3: IRLML6344TRPBFee, PyroChannel:SOT-23, F.Cu at (179.3, 110.7)
- added Q4: IRLML6344TRPBFee, PyroChannel:SOT-23, F.Cu at (199.1, 98.0)
- added Q5: IRLML6344TRPBFee, PyroChannel:SOT-23, F.Cu at (203.5, 98.0)
- added Q6: IRLML6344TRPBFee, PyroChannel:SOT-23, F.Cu at (168.9, 126.4)
- added Q7: IRLML6344TRPBFee, PyroChannel:SOT-23, F.Cu at (164.4, 126.4)
- added Q8: IRLML6344TRPBFee, PyroChannel:SOT-23, F.Cu at (188.8, 100.4)
- added Q9: IRLML6344TRPBFee, PyroChannel:SOT-23, F.Cu at (184.4, 100.4)
- added R1: 330, Resistor_SMD:R_0603_1608Metric, F.Cu at (112.4, 125.7)
- added R10: 10k, Resistor_SMD:R_0402_1005Metric, F.Cu at (187.3, 114.0)
- added R11: 10k, Resistor_SMD:R_0402_1005Metric, F.Cu at (201.2, 101.2)
- added R12: 3.3, Resistor_SMD:R_0402_1005Metric, F.Cu at (207.0, 101.2)
- added R13: 10k, Resistor_SMD:R_0402_1005Metric, F.Cu at (204.1, 101.2)
- added R14: 10k, Resistor_SMD:R_0402_1005Metric, F.Cu at (198.3, 101.2)
- added R15: 10k, Resistor_SMD:R_0402_1005Metric, F.Cu at (163.6, 129.6)
- added R16: 3.3, Resistor_SMD:R_0402_1005Metric, F.Cu at (166.6, 129.6)
- added R17: 10k, Resistor_SMD:R_0402_1005Metric, F.Cu at (169.5, 129.6)
- added R18: 10k, Resistor_SMD:R_0402_1005Metric, F.Cu at (172.4, 129.6)
- added R19: 95.5k, Resistor_SMD:R_0402_1005Metric, F.Cu at (204.0, 87.0)
- added R2: 330, Resistor_SMD:R_0603_1608Metric, F.Cu at (118.4, 121.3)
- added R20: 47k, Resistor_SMD:R_0402_1005Metric, F.Cu at (204.0, 89.0)
- added R21: 5k, Resistor_SMD:R_0402_1005Metric, F.Cu at (155.4, 121.4)
- added R22: 5k, Resistor_SMD:R_0402_1005Metric, F.Cu at (155.4, 117.4)
- added R23: 10k, Resistor_SMD:R_0402_1005Metric, F.Cu at (192.3, 103.7)
- added R24: 3.3, Resistor_SMD:R_0402_1005Metric, F.Cu at (189.4, 103.7)
- added R25: 10k, Resistor_SMD:R_0402_1005Metric, F.Cu at (186.5, 103.7)
- added R26: 10k, Resistor_SMD:R_0402_1005Metric, F.Cu at (183.6, 103.7)
- added R27: 180, Resistor_SMD:R_0402_1005Metric, F.Cu at (104.6, 121.1)
- added R28: 270, Resistor_SMD:R_0402_1005Metric, F.Cu at (155.4, 123.3)
- added R29: 270, Resistor_SMD:R_0402_1005Metric, F.Cu at (153.7, 126.8)
- added R3: 330, Resistor_SMD:R_0603_1608Metric, F.Cu at (116.4, 125.7)
- added R4: 10k, Resistor_SMD:R_0402_1005Metric, F.Cu at (168.1, 115.4)
- added R5: 10k, Resistor_SMD:R_0402_1005Metric, F.Cu at (104.6, 79.8)
- added R6: 10k, Resistor_SMD:R_0402_1005Metric, F.Cu at (197.7, 116.4)
- added R7: 10k, Resistor_SMD:R_0402_1005Metric, F.Cu at (178.6, 114.0)
- added R8: 3.3, Resistor_SMD:R_0402_1005Metric, F.Cu at (181.5, 114.0)
- added R9: 10k, Resistor_SMD:R_0402_1005Metric, F.Cu at (184.4, 114.0)
- added U1: STM32F423RHTx, Package_QFP:LQFP-64_10x10mm_P0.5mm, F.Cu at (103.3, 101.4)
- added U2: ST_H3LIS331DL, Accelerometer_Breakout:TFLGA-16_3x3mm, F.Cu at (194.1, 110.0)
- added U3: WB_W25N512GVPIT, FHSD:SON127P800X600X80-9N, F.Cu at (171.5, 91.3)
- added U4: FT232RL-REEL, Footrpint Library:SOP65P780X200-28N, F.Cu at (149.1, 120.1)
- added U5: OP179GRT, Package_TO_SOT_SMD:SOT-23-5, F.Cu at (200.1, 88.3)
- added U6: TE_MS560702BA03-50, Barometer:MS560702BA03-50, F.Cu at (169.2, 101.6)
- added U7: ST_LSM9DS1, Package_LGA:LGA-24L_3x3.5mm_P0.43mm, F.Cu at (185.4, 88.4)
- added USB1: USB_C_Receptacle, Connector_USB:USB_C_Receptacle_GCT_USB4085, F.Cu at (135.5, 116.0)
- added Y1: ECS-260-8-36B-CKY-TR, NOVA MCU (STM):ECX-2236B, F.Cu at (163.3, 118.2)
- added Y2: JTX310, NOVA MCU (STM):JTX310, F.Cu at (163.2, 115.8)
- added xt1: Conn_01x02, Connector_AMASS:AMASS_XT30PW-M_1x02_P2.50mm_Horizontal, F.Cu at (145.5, 80.9)

Commit message: Fixing out some layouts
Parts:
- removed USB1: USB_C_Receptacle, Connector_USB:USB_C_Receptacle_GCT_USB4085
- added J7: USB_C_Receptacle_USB2.0, Connector_USB:USB_C_Receptacle_GCT_USB4085, F.Cu at (156.1, 175.2)
- moved R5 159.7 mm to (262.3, 54.4)
- moved J1 150.0 mm to (23.9, 46.1)
- moved C10 146.5 mm to (47.1, 54.4)
- moved C11 146.5 mm to (50.0, 56.4)
- moved C13 146.5 mm to (47.1, 58.4)
- moved C14 146.5 mm to (50.0, 54.4)
- moved C15 146.5 mm to (47.1, 56.4)
- moved C6 146.5 mm to (55.8, 54.4)
- moved C7 146.5 mm to (52.9, 56.4)
- moved C8 146.5 mm to (50.0, 58.4)
- moved C9 146.5 mm to (52.9, 54.4)
- moved C24 144.2 mm to (259.9, 63.6)
- moved J6 132.4 mm to (222.5, 99.2), turned to 270 degrees
- moved C21 130.9 mm to (40.2, 87.9)
- moved C18 130.9 mm to (43.1, 89.1)
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
Commit message: Began Laying out sub modules
Parts:
- R12, R16, R24, R8: footprint Resistor_SMD:R_0402_1005Metric -> Package_TO_SOT_SMD:TO-252-2
- moved C2 219.5 mm to (295.9, 111.4), turned to 270 degrees
- moved 3v3Reg1 217.5 mm to (290.4, 111.9)
- moved C1 213.5 mm to (285.0, 113.7), turned to 270 degrees
- moved D3 212.0 mm to (282.6, 115.2), turned to 90 degrees
- moved xt1 209.6 mm to (270.1, 118.0)
- moved D4 202.8 mm to (279.1, 114.2)
- moved D2 160.9 mm to (116.5, 20.7)
- moved BZ1 160.9 mm to (109.4, 24.0)
- moved Q10 160.9 mm to (116.4, 24.5)
- moved R27 160.9 mm to (120.4, 20.2)
- moved D1 157.7 mm to (90.5, 23.7)
- moved R1 157.7 mm to (89.5, 27.1)
- moved R3 157.7 mm to (93.5, 27.1)
- moved R2 157.7 mm to (95.5, 22.7)
- moved R19 155.7 mm to (129.6, 23.0)
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Connections:
- J5 pad 2: GND -> Net-(C24-Pad1)
- J5 pad 4: GND -> Net-(C24-Pad1)
- J6 pad 2: GND -> Net-(C24-Pad1)
- J6 pad 4: GND -> Net-(C24-Pad1)

Commit message: More Layout
Parts:
- C10, C11, C12, C13, C14, C15, C16, C17, C18, C19, C20, C21, C22, C23, C25, C27, C3, C5, C6, C7, C8, C9, Q2, Q3, Q4, Q5, Q6, Q7, Q8, Q9, R10, R11, R13, R14, R15, R17, R18, R21, R22, R23, R25, R26, R4, R7, R9, Y1, Y2: moved to B.Cu
- Micro_SD1: footprint Connector_Card:microSD_HC_Wuerth_693072010801 -> Connector_Card:microSD_HC_Molex_104031-0811
- moved H1 173.4 mm to (209.8, 105.2)
- moved H2 173.0 mm to (217.0, 97.4)
- moved H3 173.0 mm to (217.0, 105.4)
- moved H4 173.0 mm to (209.4, 97.4)
- moved C2 129.9 mm to (166.3, 102.1), turned to 90 degrees
- moved C20 124.4 mm to (164.9, 61.6), turned to 225 degrees
- moved R4 124.2 mm to (166.3, 66.3), turned to 135 degrees
- moved Y1 123.7 mm to (167.5, 63.6), turned to 135 degrees
- moved C19 123.2 mm to (168.1, 65.3), turned to 45 degrees
- moved 3v3Reg1 121.7 mm to (169.4, 98.8), turned to 180 degrees
- moved C26 120.3 mm to (131.7, 53.9)
- moved U3 120.3 mm to (134.5, 60.6)
- moved D3 119.4 mm to (164.9, 95.5), turned to 0 degrees
- moved C21 118.9 mm to (161.2, 55.4), turned to 135 degrees
- moved Y2 118.6 mm to (161.1, 52.7), turned to 315 degrees
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Connections:
- J3 pad 10: +BATT -> (no net)
- J3 pad 4: /MOSI -> (no net)
- J3 pad 5: /MISO -> /MOSI
- J3 pad 7: (no net) -> /MISO
- J3 pad 9: (no net) -> +BATT
- J5 pad 1: /Pyro Channels/PYRO1 -> /Pyro Channels/PYRO2
- J5 pad 3: /Pyro Channels/PYRO2 -> /Pyro Channels/PYRO1
- J6 pad 1: /Pyro Channels/PYRO3 -> /Pyro Channels/PYRO4
- J6 pad 3: /Pyro Channels/PYRO4 -> /Pyro Channels/PYRO3
- U1 pad 26: (no net) -> /FL_CS
- U3 pad 1: (no net) -> /FL_CS
Routing:
- net Net-(C24-Pad1): track 0.00 -> 58.9 mm
- net GND: track 0.00 -> 47.8 mm, vias 0 -> 20
- net +3V3: track 0.00 -> 28.8 mm, vias 0 -> 7
- net +BATT: track 0.00 -> 28.1 mm
- net /Pyro Channels/PYRO3: track 0.00 -> 16.6 mm
- net /Pyro Channels/PYRO1: track 0.00 -> 16.5 mm
- net /Pyro Channels/PYRO4: track 0.00 -> 15.9 mm
- net /Pyro Channels/PYRO2: track 0.00 -> 15.8 mm
- net Net-(3v3Reg1-Pad3): track 0.00 -> 11.0 mm
- net /CLOCKOUT: track 0.00 -> 9.36 mm, vias 0 -> 1
- net /Pyro Channels/Arm Schematic/FireOut: track 0.00 -> 7.35 mm
- net Net-(Q4-Pad2): track 0.00 -> 7.20 mm, vias 0 -> 1
- net /32CLOCKOUT: track 0.00 -> 7.08 mm, vias 0 -> 1
- net Net-(Q2-Pad2): track 0.00 -> 6.81 mm, vias 0 -> 1
- net /FIRE3: track 0.00 -> 6.78 mm
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Other:
- net class High-Current added: clearance 0.15, trace_width 1, via_dia 0.8, via_drill 0.4
- net class Pyro removed
- net class Signals removed
- net class Standard added: clearance 0.15, trace_width 0.25, via_dia 0.6, via_drill 0.3
