File: Electrical/Nova/PyroLogic1.sch (KiCad schematic (older format))
At the start: 5 parts, among them Q1 Q_NMOS_DGS, Q2 Q_NMOS_DGS

Commit message: Assigned footprints to several components
Parts:
- Q1, Q2: footprint (none) -> Package_TO_SOT_SMD:SOT-23-6_Handsoldering
- R10, R8, R9: footprint (none) -> Resistor_SMD:R_0805_2012Metric_Pad1.15x1.40mm_HandSolder
Changed lines of the file:
@@
 F 0 "Q1" H 5354 2646 50  0000 L CNN
 F 1 "Q_NMOS_DGS" H 5354 2555 50  0000 L CNN
-F 2 "" H 5350 2700 50  0001 C CNN
+F 2 "Package_TO_SOT_SMD:SOT-23-6_Handsoldering" H 5350 2700 50  0001 C CNN
 F 3 "~" H 5150 2600 50  0001 C CNN
 	1    5150 2600
@@
 F 0 "Q2" H 5354 3646 50  0000 L CNN
 F 1 "Q_NMOS_DGS" H 5354 3555 50  0000 L CNN
-F 2 "" H 5350 3700 50  0001 C CNN
+F 2 "Package_TO_SOT_SMD:SOT-23-6_Handsoldering" H 5350 3700 50  0001 C CNN
 F 3 "~" H 5150 3600 50  0001 C CNN
 	1    5150 3600
@@
 F 0 "R10" H 5318 3146 50  0000 L CNN
 F 1 "3.3" H 5318 3055 50  0000 L CNN
-F 2 "" V 5290 3090 50  0001 C CNN
+F 2 "Resistor_SMD:R_0805_2012Metric_Pad1.15x1.40mm_HandSolder" V 5290 3090 50  0001 C CNN
 F 3 "~" H 5250 3100 50  0001 C CNN
 	1    5250 3100
@@
 F 0 "R8" H 4818 2996 50  0000 L CNN
 F 1 "10k" H 4818 2905 50  0000 L CNN
-F 2 "" V 4790 2940 50  0001 C CNN
+F 2 "Resistor_SMD:R_0805_2012Metric_Pad1.15x1.40mm_HandSolder" V 4790 2940 50  0001 C CNN
 F 3 "~" H 4750 2950 50  0001 C CNN
 	1    4750 2950
@@
 F 0 "R9" H 4818 3996 50  0000 L CNN
 F 1 "10k" H 4818 3905 50  0000 L CNN
-F 2 "" V 4790 3940 50  0001 C CNN
+F 2 "Resistor_SMD:R_0805_2012Metric_Pad1.15x1.40mm_HandSolder" V 4790 3940 50  0001 C CNN
 F 3 "~" H 4750 3950 50  0001 C CNN
 	1    4750 3950

Commit message: Began Layout of Nova Rev 2 PCB Updated Version
Parts:
- Q1, Q2: symbol Device:Q_NMOS_DGS -> MOSFET:Q_NMOS_DGS
Changed lines of the file:
@@
 $EndDescr
 $Comp
-L Device:Q_NMOS_DGS Q1
+L MOSFET:Q_NMOS_DGS Q1
 U 1 1 617E0250
 P 5150 2600
@@
 $EndComp
 $Comp
-L Device:Q_NMOS_DGS Q2
+L MOSFET:Q_NMOS_DGS Q2
 U 1 1 617E0251
 P 5150 3600

Commit message: Silkscreen Cleanup
Parts:
- Q1, Q2: symbol MOSFET:Q_NMOS_DGS -> Nova-rescue:Q_NMOS_DGS-MOSFET
Changed lines of the file:
@@
 $EndDescr
 $Comp
-L MOSFET:Q_NMOS_DGS Q1
+L Nova-rescue:Q_NMOS_DGS-MOSFET Q1
 U 1 1 617E0250
 P 5150 2600
@@
 AR Path="/5F448D4B/617C2A68/617E0250" Ref="Q?"  Part="1"
 AR Path="/5F448D4B/617C3265/617E0250" Ref="Q?"  Part="1"
+AR Path="/617E0250" Ref="Q1"  Part="1"
 F 0 "Q1" H 5354 2646 50  0000 L CNN
 F 1 "Q_NMOS_DGS" H 5354 2555 50  0000 L CNN
@@
 $EndComp
 $Comp
-L MOSFET:Q_NMOS_DGS Q2
+L Nova-rescue:Q_NMOS_DGS-MOSFET Q2
 U 1 1 617E0251
 P 5150 3600
@@
 AR Path="/5F448D4B/617C2A68/617E0251" Ref="Q?"  Part="1"
 AR Path="/5F448D4B/617C3265/617E0251" Ref="Q?"  Part="1"
+AR Path="/617E0251" Ref="Q2"  Part="1"
 F 0 "Q2" H 5354 3646 50  0000 L CNN
 F 1 "Q_NMOS_DGS" H 5354 3555 50  0000 L CNN
