File: Electrical/Nova/PyroLogic3.sch (KiCad schematic (older format))
At the start: 5 parts, among them Q5 Q_NMOS_DGS, Q6 Q_NMOS_DGS

Commit message: Assigned footprints to several components
Parts:
- Q5, Q6: footprint (none) -> Package_TO_SOT_SMD:SOT-23-6_Handsoldering
- R14, R15, R16: footprint (none) -> Resistor_SMD:R_0805_2012Metric_Pad1.15x1.40mm_HandSolder
Changed lines of the file:
@@
 F 0 "Q5" H 5354 2646 50  0000 L CNN
 F 1 "Q_NMOS_DGS" H 5354 2555 50  0000 L CNN
-F 2 "" H 5350 2700 50  0001 C CNN
+F 2 "Package_TO_SOT_SMD:SOT-23-6_Handsoldering" H 5350 2700 50  0001 C CNN
 F 3 "~" H 5150 2600 50  0001 C CNN
 	1    5150 2600
@@
 F 0 "Q6" H 5354 3646 50  0000 L CNN
 F 1 "Q_NMOS_DGS" H 5354 3555 50  0000 L CNN
-F 2 "" H 5350 3700 50  0001 C CNN
+F 2 "Package_TO_SOT_SMD:SOT-23-6_Handsoldering" H 5350 3700 50  0001 C CNN
 F 3 "~" H 5150 3600 50  0001 C CNN
 	1    5150 3600
@@
 F 0 "R16" H 5318 3146 50  0000 L CNN
 F 1 "3.3" H 5318 3055 50  0000 L CNN
-F 2 "" V 5290 3090 50  0001 C CNN
+F 2 "Resistor_SMD:R_0805_2012Metric_Pad1.15x1.40mm_HandSolder" V 5290 3090 50  0001 C CNN
 F 3 "~" H 5250 3100 50  0001 C CNN
 	1    5250 3100
@@
 F 0 "R14" H 4818 2996 50  0000 L CNN
 F 1 "10k" H 4818 2905 50  0000 L CNN
-F 2 "" V 4790 2940 50  0001 C CNN
+F 2 "Resistor_SMD:R_0805_2012Metric_Pad1.15x1.40mm_HandSolder" V 4790 2940 50  0001 C CNN
 F 3 "~" H 4750 2950 50  0001 C CNN
 	1    4750 2950
@@
 F 0 "R15" H 4818 3996 50  0000 L CNN
 F 1 "10k" H 4818 3905 50  0000 L CNN
-F 2 "" V 4790 3940 50  0001 C CNN
+F 2 "Resistor_SMD:R_0805_2012Metric_Pad1.15x1.40mm_HandSolder" V 4790 3940 50  0001 C CNN
 F 3 "~" H 4750 3950 50  0001 C CNN
 	1    4750 3950

Commit message: Began Layout of Nova Rev 2 PCB Updated Version
Parts:
- Q5, Q6: symbol Device:Q_NMOS_DGS -> MOSFET:Q_NMOS_DGS
Changed lines of the file:
@@
 $EndDescr
 $Comp
-L Device:Q_NMOS_DGS Q?
+L MOSFET:Q_NMOS_DGS Q?
 U 1 1 617DF88C
 P 5150 2600
@@
 $EndComp
 $Comp
-L Device:Q_NMOS_DGS Q?
+L MOSFET:Q_NMOS_DGS Q?
 U 1 1 617DF88D
 P 5150 3600

Commit message: Silkscreen Cleanup
Parts:
- Q5, Q6: symbol MOSFET:Q_NMOS_DGS -> Nova-rescue:Q_NMOS_DGS-MOSFET
Changed lines of the file:
@@
 $EndDescr
 $Comp
-L MOSFET:Q_NMOS_DGS Q?
+L Nova-rescue:Q_NMOS_DGS-MOSFET Q?
 U 1 1 617DF88C
 P 5150 2600
@@
 AR Path="/5F448D4B/617C2A68/617DF88C" Ref="Q5"  Part="1"
 AR Path="/5F448D4B/617C3265/617DF88C" Ref="Q?"  Part="1"
+AR Path="/617DF88C" Ref="Q5"  Part="1"
 F 0 "Q5" H 5354 2646 50  0000 L CNN
 F 1 "Q_NMOS_DGS" H 5354 2555 50  0000 L CNN
@@
 $EndComp
 $Comp
-L MOSFET:Q_NMOS_DGS Q?
+L Nova-rescue:Q_NMOS_DGS-MOSFET Q?
 U 1 1 617DF88D
 P 5150 3600
@@
 AR Path="/5F448D4B/617C2A68/617DF88D" Ref="Q6"  Part="1"
 AR Path="/5F448D4B/617C3265/617DF88D" Ref="Q?"  Part="1"
+AR Path="/617DF88D" Ref="Q6"  Part="1"
 F 0 "Q6" H 5354 3646 50  0000 L CNN
 F 1 "Q_NMOS_DGS" H 5354 3555 50  0000 L CNN
