File: Electrical/Nova/Nova.kicad_sch (KiCad schematic)
At the start: 13 parts, among them J2 Conn_02x04_Counter_Clockwise, U1 STM32F411CEUx

Commit message: Working on re-routing
Connections:
- net INT1 is gone; now on net ACCEL_INT1: U1.19 (PB1)
- net INT2 is gone; now on net ACCEL_INT2: U1.20 (PB2)
Changed lines of the file:
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@@
     (stroke (width 0) (type default) (color 0 0 0 0))
   )
-  (polyline (pts (xy 39.37 73.66) (xy 85.09 73.66))
+  (polyline (pts (xy 39.37 74.93) (xy 85.09 74.93))
     (stroke (width 0) (type default) (color 0 0 0 0))
   )
@@
     (stroke (width 0) (type default) (color 0 0 0 0))
   )
-  (polyline (pts (xy 39.37 19.05) (xy 39.37 73.66))
+  (polyline (pts (xy 39.37 19.05) (xy 39.37 74.93))
     (stroke (width 0) (type default) (color 0 0 0 0))
   )
@@
     (stroke (width 0) (type default) (color 0 0 0 0))
   )
-  (polyline (pts (xy 85.09 73.66) (xy 85.09 19.05))
+  (polyline (pts (xy 85.09 74.93) (xy 85.09 19.05))
     (stroke (width 0) (type default) (color 0 0 0 0))
   )
@@
     (effects (font (size 2.0066 2.0066)) (justify left bottom))
   )
-  (text "MCU PERIPHERALS\n\n" (at 48.26 80.01 0)
+  (text "MCU PERIPHERALS\n\n" (at 48.26 81.28 0)
     (effects (font (size 2.0066 2.0066)) (justify left bottom))
   )
@@
     (effects (font (size 1.27 1.27)) (justify left bottom))
   )
-  (label "INT1" (at 46.99 140.97 180)
+  (label "ACCEL_INT1" (at 46.99 140.97 180)
     (effects (font (size 1.27 1.27)) (justify right bottom))
   )
@@
     (effects (font (size 1.27 1.27)) (justify right bottom))
   )
-  (label "INT2" (at 46.99 143.51 180)
-    (effects (font (size 1.27 1.27)) (justify right bottom))
-  )
+  (label "ACCEL_INT2" (at 46.99 143.51 180)
+    (effects (font (size 1.27 1.27)) (justify right bottom))
+  )

Commit message: Updated cryatal pins to reflect datasheet, changed vcap to reflect datasheet
Parts:
- U1: footprint Package_DFN_QFN:QFN-48-1EP_7x7mm_P0.5mm_EP5.6x5.6mm -> STMf411:STM32F411CEU6
Changed lines of the file:
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@@
     (property "Reference" "U1" (id 0) (at 66.04 90.17 0))
     (property "Value" "STM32F411CEUx" (id 1) (at 66.04 87.63 0))
-    (property "Footprint" "Package_DFN_QFN:QFN-48-1EP_7x7mm_P0.5mm_EP5.6x5.6mm" (id 2) (at 50.8 176.53 0)
+    (property "Footprint" "STMf411:STM32F411CEU6" (id 2) (at 50.8 176.53 0)
       (effects (font (size 1.27 1.27)) (justify right) hide)
     )
@@
       (reference "#PWR0163") (unit 1) (value "GND") (footprint "")
     )
+    (path "/00000000-0000-0000-0000-00005f319c9c/fc37719f-2e63-4176-896a-7a97074d32ca"
+      (reference "#PWR0164") (unit 1) (value "GND") (footprint "")
+    )
+    (path "/00000000-0000-0000-0000-00005f319c9c/98bafe4f-e043-4d95-9cbb-e623ecfee013"
+      (reference "#PWR0165") (unit 1) (value "GND") (footprint "")
+    )
     (path "/00000000-0000-0000-0000-000061c94220"
       (reference "BOOT1") (unit 1) (value "SW_Push") (footprint "NOVA MCU (STM):KSR223GLFG")
@@
     )
     (path "/00000000-0000-0000-0000-00005f319c9c/00000000-0000-0000-0000-000061c6928d"
-      (reference "C7") (unit 1) (value "1.5pF") (footprint "Capacitor_SMD:C_0402_1005Metric")
+      (reference "C7") (unit 1) (value "8pF") (footprint "Capacitor_SMD:C_0402_1005Metric")
     )
     (path "/00000000-0000-0000-0000-00005f319c9c/00000000-0000-0000-0000-000061c69a59"
-      (reference "C8") (unit 1) (value "1.5pF") (footprint "Capacitor_SMD:C_0402_1005Metric")
+      (reference "C8") (unit 1) (value "8pF") (footprint "Capacitor_SMD:C_0402_1005Metric")
     )
     (path "/00000000-0000-0000-0000-00005f319c9c/00000000-0000-0000-0000-000061c69d3a"
@@
     )
     (path "/00000000-0000-0000-0000-00005f3189b2/00000000-0000-0000-0000-000061bc2f35"
-      (reference "C10") (unit 1) (value "2.2uF") (footprint "Capacitor_SMD:C_0402_1005Metric")
+      (reference "C10") (unit 1) (value "4.7uF") (footprint "Capacitor_SMD:C_0402_1005Metric")
     )
     (path "/00000000-0000-0000-0000-00005f319c9c/00000000-0000-0000-0000-000061c69e7c"
@@
     )
     (path "/00000000-0000-0000-0000-00005f3b5c2e/00000000-0000-0000-0000-00005f06d2e9"
-      (reference "C26") (unit 1) (value "0.1uF") (footprint "Capacitor_SMD:C_0402_1005Metric")
+      (reference "C26") (unit 1) (value "100nF") (footprint "Capacitor_SMD:C_0402_1005Metric")
     )
     (path "/00000000-0000-0000-0000-00005f319d4b/00000000-0000-0000-0000-0000607642f6"
@@
     )
     (path "/00000000-0000-0000-0000-00005f319d4b/00000000-0000-0000-0000-00005f9b6a21"
-      (reference "R21") (unit 1) (value "5k") (footprint "Resistor_SMD:R_0402_1005Metric")
+      (reference "R21") (unit 1) (value "5k1") (footprint "Resistor_SMD:R_0402_1005Metric")
     )
     (path "/00000000-0000-0000-0000-00005f319d4b/00000000-0000-0000-0000-00005f9b6a27"
-      (reference "R22") (unit 1) (value "5k") (footprint "Resistor_SMD:R_0402_1005Metric")
+      (reference "R22") (unit 1) (value "5k1") (footprint "Resistor_SMD:R_0402_1005Metric")
     )
     (path "/00000000-0000-0000-0000-00005f448d4b/00000000-0000-0000-0000-0000617c3265/00000000-0000-0000-0000-0000617e0252"
@@
     )
     (path "/00000000-0000-0000-0000-0000615ccc8f"
-      (reference "U1") (unit 1) (value "STM32F411CEUx") (footprint "Package_DFN_QFN:QFN-48-1EP_7x7mm_P0.5mm_EP5.6x5.6mm")
+      (reference "U1") (unit 1) (value "STM32F411CEUx") (footprint "STMf411:STM32F411CEU6")
     )
     (path "/00000000-0000-0000-0000-00005f46051d/00000000-0000-0000-0000-00005f0cd93e"
